File: EL - Electrical/Autre/Passage de vitesse/Optimus/Hardware/shield passage vitesse.brd (EAGLE design)
At the start: 69.2 x 53.4 mm, 37 parts, among them J1 22-05-7078-07, J2 22-05-7038-03, J3 22-05-7028-02, J5 22-05-7028-02, J6 22-05-7028-02, Q1 2N7000, Q2 2N7000, Q3 2N7000, Q4 2N7000, Q5 2N7000

Commit message: Carte Passage vitesse
Parts:
- removed J1: 22-05-7078-07, EP_molex_6410_7395:7395-07
- removed J2: 22-05-7038-03, EP_molex_6410_7395:7395-03
- removed J3, J6: 22-05-7028-02, EP_molex_6410_7395:7395-02
- added ALIM_ARDUINO, CONN_ECU_(DTA): 22-05-7028-02, EP_molex_6410_7395:7395-02
- added CONN_MOTOR: 22-05-7078-07, EP_molex_6410_7395:7395-07
- added CONN_PALETTE: 22-05-7038-03, EP_molex_6410_7395:7395-03
- moved R15 118.6 mm to (14.1, 45.5)
- moved R17 115.3 mm to (14.2, 41.1)
- moved R13 114.4 mm to (57.3, 28.8)
- moved R14 108.4 mm to (57.3, 26.5), turned to 180 degrees
- moved R5 102.9 mm to (37.5, 38.0), turned to 180 degrees
- moved R12 102.7 mm to (57.3, 33.7), turned to 180 degrees
- moved R6 101.7 mm to (35.9, 35.8), turned to 180 degrees
- moved R1 101.7 mm to (37.5, 31.4), turned to 180 degrees
- moved R11 101.5 mm to (57.3, 31.4)
- moved Q2 100.9 mm to (44.8, 31.4)
- moved R2 96.7 mm to (35.9, 29.2), turned to 180 degrees
- moved Q1 93.7 mm to (44.8, 38.0)
- moved R7 91.3 mm to (37.5, 16.4), turned to 180 degrees
- moved R3 89.8 mm to (37.5, 23.7), turned to 180 degrees
- moved Q3 89.0 mm to (44.8, 23.7)
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- renumbered DIGITALIN0-7 to DIGITALIN0_7, DIGITALIN8-13 to DIGITALIN8_13
Connections:
- net 12V: now also ALIM_ARDUINO.2; no longer J6.2
- net 5V: now also CONN_PALETTE.2; no longer J2.2
- net GND: now also ALIM_ARDUINO.1, DIGITALIN8_13.2; no longer DIGITALIN8_13.7, J6.1
- net IN0_12V: now also CONN_MOTOR.7; no longer J1.7
- net IN1_12V: now also CONN_MOTOR.6; no longer J1.6
- net OUT0_12V: now also CONN_MOTOR.5, Q1.3; no longer J1.5, Q3.3
- net OUT0_5V: now also DIGITALIN0_7.1, Q1.1; no longer DIGITALIN8_13.2, Q3.1
- net OUT1_12V: now also CONN_MOTOR.4, Q2.3; no longer J1.4, Q1.3
- net OUT1_5V: now also DIGITALIN0_7.2, Q2.1; no longer DIGITALIN8_13.1, Q1.1
- net OUT2_12V: now also CONN_MOTOR.3, Q3.3; no longer J1.3, Q2.3
- net OUT2_5V: now also DIGITALIN0_7.3, Q3.1; no longer DIGITALIN0_7.8, Q2.1
- net OUT3_12V: now also CONN_MOTOR.2; no longer J1.2
- net OUT3_5V: now also DIGITALIN0_7.4; no longer DIGITALIN0_7.7
- net OUT4_12V: now also CONN_MOTOR.1; no longer J1.1
- net OUT4_5V: now also DIGITALIN0_7.5; no longer DIGITALIN0_7.6
- net PALETTE_DROITE: now also CONN_PALETTE.3, DIGITALIN8_13.8; no longer DIGITALIN0_7.1, J2.3
- net PALETTE_GAUCHE: now also CONN_PALETTE.1, DIGITALIN8_13.7; no longer DIGITALIN0_7.2, J2.1
- net SHIFT_CUT: now also CONN_ECU_(DTA).2, DIGITALIN0_7.8; no longer DIGITALIN0_7.5, J3.2
- net SHIFT_POT: now also CONN_ECU_(DTA).1, DIGITALIN0_7.7; no longer DIGITALIN0_7.4, J3.1
Routing:
- net 5V: track 0.00 -> 133.1 mm
- net 12V: track 0.00 -> 82.2 mm
- net GND: track 0.00 -> 80.8 mm
- net OUT4_5V: track 0.00 -> 58.7 mm
- net OUT3_5V: track 0.00 -> 52.3 mm
- net SHIFT_POT: track 0.00 -> 49.9 mm
- net SHIFT_CUT: track 0.00 -> 47.0 mm
- net OUT2_5V: track 0.00 -> 45.3 mm
- net PALETTE_DROITE: track 0.00 -> 42.2 mm
- net PALETTE_GAUCHE: track 0.00 -> 35.9 mm
- net OUT0_12V: track 0.00 -> 22.4 mm
- net OUT1_5V: track 0.00 -> 20.5 mm
- net OUT1_12V: track 0.00 -> 17.9 mm
- net OUT2_12V: track 0.00 -> 12.3 mm
- net OUT4_12V: track 0.00 -> 11.8 mm
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