File: EL - Electrical/Autre/Passage de vitesse/Optimus/Hardware/shield passage vitesse.brd (EAGLE design)
At the start: 69.2 x 53.4 mm, 37 parts, among them J5 22-05-7028-02, Q1 2N7000, Q2 2N7000, Q3 2N7000, Q4 2N7000, Q5 2N7000

Commit message: plein de choses
Parts:
- C4, C5: value 0.33u -> 0.33uF
- moved C5 6.48 mm to (18.0, 37.8)
- renumbered CONN_ECU_(DTA) to ECU, CONN_PALETTE to PALETTE, J5 to BATTERIE
Routing:
- net GND: track 100.9 -> 0.00 mm
- net 5V: track 143.4 -> 131.8 mm
- net SHIFT_CUT: track 45.4 -> 46.7 mm
Other:
- outline, holes or cut-outs redrawn
