File: EL - Electrical/Autre/BSPD/BSPD.brd (EAGLE design)
At the start: 160 x 100 mm, 8 parts, among them IC1 4013N, IC3 LM2901N

Commit message: et hop je dépasse benji
Parts:
- moved IC1 123.2 mm to (100.3, 87.6), turned to 90 degrees
Changed lines of the file:
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@@
 <attribute name="VALUE" x="88.265" y="42.291" size="1.27" layer="27" ratio="10" rot="R270"/>
 </element>
-<element name="IC1" library="40xx" library_urn="urn:adsk.eagle:library:80" package="DIL14" package3d_urn="urn:adsk.eagle:package:820/2" value="4013N" x="17.78" y="-3.81" smashed="yes">
-<attribute name="NAME" x="8.509" y="-6.858" size="1.27" layer="25" ratio="10" rot="R90"/>
-<attribute name="VALUE" x="11.049" y="-4.445" size="1.27" layer="27" ratio="10"/>
+<element name="IC1" library="40xx" library_urn="urn:adsk.eagle:library:80" package="DIL14" package3d_urn="urn:adsk.eagle:package:820/2" value="4013N" x="100.33" y="87.63" smashed="yes" rot="R90">
+<attribute name="NAME" x="103.378" y="78.359" size="1.27" layer="25" ratio="10" rot="R180"/>
+<attribute name="VALUE" x="100.965" y="80.899" size="1.27" layer="27" ratio="10" rot="R90"/>
 </element>
 </elements>
@@
 <wire x1="67.31" y1="38.1" x2="85.09" y2="33.02" width="0" layer="19" extent="1-1"/>
 <wire x1="67.31" y1="40.64" x2="67.31" y2="38.1" width="0" layer="19" extent="1-1"/>
-<wire x1="20.32" y1="-7.62" x2="67.31" y2="38.1" width="0" layer="19" extent="1-1"/>
+<wire x1="104.14" y1="90.17" x2="67.31" y2="38.1" width="0" layer="19" extent="1-1"/>
 </signal>
 <signal name="N$2">
@@
 <wire x1="45.72" y1="21.59" x2="85.09" y2="27.94" width="0" layer="19" extent="1-1"/>
 <wire x1="40.64" y1="21.59" x2="45.72" y2="21.59" width="0" layer="19" extent="1-1"/>
-<wire x1="22.86" y1="0" x2="40.64" y2="21.59" width="0" layer="19" extent="1-1"/>
+<wire x1="96.52" y1="92.71" x2="40.64" y2="21.59" width="0" layer="19" extent="1-1"/>
 </signal>
 <signal name="N$4">
@@
 <contactref element="IC1" pad="11"/>
 <contactref element="IC3" pad="1"/>
-<wire x1="17.78" y1="0" x2="85.09" y2="43.18" width="0" layer="19" extent="1-1"/>
+<wire x1="96.52" y1="87.63" x2="85.09" y2="43.18" width="0" layer="19" extent="1-1"/>
 </signal>
 <signal name="N$6">
 <contactref element="IC3" pad="2"/>
 <contactref element="IC1" pad="3"/>
-<wire x1="15.24" y1="-7.62" x2="85.09" y2="40.64" width="0" layer="19" extent="1-1"/>
+<wire x1="104.14" y1="85.09" x2="85.09" y2="40.64" width="0" layer="19" extent="1-1"/>
 </signal>
 </signals>

Commit message: BSPD
Connections:
- new net 5V: R2.2
- new net N$7: R1.2
Changed lines of the file:
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@@
 <wire x1="104.14" y1="85.09" x2="85.09" y2="40.64" width="0" layer="19" extent="1-1"/>
+</signal>
+<signal name="5V">
+<contactref element="R2" pad="2"/>
+</signal>
+<signal name="N$7">
+<contactref element="R1" pad="2"/>
 </signal>
 </signals>

Commit message: de l'élec
Parts:
- added C3, C4: 100uF, rcl:C025-025X050
- added D1: 1N5817-B, diode:DO41-7.6
- added IC2, IC7: 4001N, 40xx:DIL14
- added IC4: LM2576T, v-reg-3:TO220-5
- added IC5: 4013N, 40xx:DIL14
- added J1: 22-05-7068-06, con-molex:7395-06
- added K1: 35701331, relay:REED
- added L1: 100uH, wurth_elektronik_passive_rev16d:WE-TI_8012
- added R5, R6: (no value), rcl:PT-10
- C1: value (none) -> 100mF
- C2: value (none) -> 500uF
- R3, R4: value (none) -> 3k
- moved IC1 155.4 mm to (-47.0, 38.1), turned to 0 degrees
- moved C2 124.9 mm to (-57.1, 58.4), turned to 0 degrees
- moved R2 121.8 mm to (-57.1, 6.35), turned to 0 degrees
- moved IC3 115.0 mm to (-25.4, 48.3), turned to 0 degrees
- moved R1 112.3 mm to (-45.7, 6.35), turned to 0 degrees
- moved C1 104.5 mm to (-50.8, 58.4)
- moved R3 90.9 mm to (-24.1, 64.8)
- moved R4 83.2 mm to (-34.3, 64.8)
Connections:
- removed net V+: IC3.3
- removed net V-: IC3.12
- removed net VDD: IC1.14
- removed net VSS: IC1.7
- new net BP: IC3.9, J1.3
- new net N$10: IC2.4, IC5.11
- new net N$11: IC7.4, R4.1
- new net N$12: IC5.13, K1.5
- new net N$13: IC3.10, R6.3
- new net N$14: IC3.8, R5.3
- new net N$15: IC2.8, IC2.9, IC3.14
- new net N$16: D1.C, IC4.2, L1.1
- new net N$17: IC2.11, IC7.1
- new net N$18: IC2.10, IC7.2
- new net N$19: IC2.3, IC2.5, IC2.6
- new net N$21: IC1.4, IC7.10
- new net N$8: IC1.13, IC2.2, IC7.8, IC7.9
- new net N$9: IC1.1, IC2.1, IC5.9
- new net OUT: J1.4, K1.7
- new net SDC: J1.5, K1.1
- new net TPS: IC3.11, J1.2
- new net TPS&BP: IC7.3, IC7.5, IC7.6, R3.1
- new net VBAT: C4.2, IC4.1, J1.1
- net 0: now also C3.1, C4.1, D1.A, IC1.10, IC1.6, IC1.7, IC1.8, IC2.7, IC3.12, IC4.3, IC4.5, IC5.10, IC5.7, IC5.8, IC7.7, J1.6, K1.3, R5.1, R6.1
- net 5V: now also C3.2, IC1.14, IC2.14, IC3.3, IC4.4, IC5.14, IC7.14, L1.2, R1.2, R5.2, R6.2
- net N$7: now also IC2.12, IC2.13, IC3.13; no longer R1.2

Commit message: élec
Parts:
- removed R1, R2, R5, R6: (no value), rcl:PT-10
- added R10, R7, R8, R9: (no value), rcl:PT-SPIN
- moved IC2 150.8 mm to (50.8, 67.3), turned to 270 degrees
- moved J1 144.0 mm to (49.5, 86.4), turned to 180 degrees
- moved IC7 142.3 mm to (45.7, 48.3), turned to 270 degrees
- moved L1 97.0 mm to (24.1, 85.1), turned to 90 degrees
- moved IC4 94.5 mm to (30.5, 85.1), turned to 90 degrees
- moved D1 92.1 mm to (47.0, 82.5)
- moved C1 87.9 mm to (35.6, 41.9), turned to 90 degrees
- moved IC5 85.4 mm to (36.8, 67.3), turned to 270 degrees
- moved C3 79.2 mm to (15.2, 67.3), turned to 90 degrees
- moved IC1 75.6 mm to (27.9, 48.3), turned to 270 degrees
- moved K1 75.2 mm to (59.7, 71.1), turned to 270 degrees
- moved R4 75.2 mm to (38.1, 44.5), turned to 270 degrees
- moved C2 72.4 mm to (15.2, 61.0), turned to 90 degrees
- moved C4 67.0 mm to (49.5, 78.7), turned to 180 degrees
- moved IC3 51.9 mm to (22.9, 67.3), turned to 270 degrees
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Connections:
- net SDC renamed SDS
- net 0: now also R10.1, R7.1, R8.1, R9.1; no longer R1.1, R2.1, R5.1, R6.1
- net 5V: now also R10.2, R7.2, R8.2, R9.2; no longer R1.2, R2.2, R5.2, R6.2
- net N$13: now also R10.3; no longer R6.3
- net N$14: now also R8.3; no longer R5.3
- net N$2: now also R7.3; no longer R1.3
- net N$4: now also R9.3; no longer R2.3
- net N$7: no longer IC3.13
Routing:
- net 0: track 0.00 -> 213.4 mm
- net 5V: track 0.00 -> 161.7 mm
- net N$8: track 0.00 -> 69.5 mm
- net N$2: track 0.00 -> 65.4 mm
- net TPS&BP: track 0.00 -> 56.3 mm
- net BP: track 0.00 -> 53.6 mm, vias 0 -> 1
- net N$15: track 0.00 -> 46.8 mm
- net N$1: track 0.00 -> 43.1 mm
- net N$9: track 0.00 -> 39.2 mm
- net N$4: track 0.00 -> 38.5 mm
- net N$13: track 0.00 -> 36.4 mm
- net N$3: track 0.00 -> 33.8 mm
- net N$5: track 0.00 -> 31.9 mm
- net N$6: track 0.00 -> 31.5 mm, vias 0 -> 1
- net TPS: track 0.00 -> 28.9 mm
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Other:
- board size 160 x 100 mm -> 54.6 x 62.9 mm
