File: EL - Electrical/Autre/BSPD/BSPD.sch (EAGLE design)
At the start: 8 parts, among them IC1 4013N, IC3 LM2901N

Commit message: et hop je dépasse benji
Other:
- moved on the sheet: C1, C2, IC1A, IC1B, IC3A, IC3B, R1, R2, R3, R4
Changed lines of the file:
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@@
 <attribute name="SHEET" x="230.505" y="5.08" size="2.54" layer="94"/>
 </instance>
-<instance part="X_1" gate="G$1" x="73.66" y="116.84" smashed="yes"/>
-<instance part="R1" gate="1" x="83.82" y="109.22" smashed="yes" rot="R180">
-<attribute name="NAME" x="81.28" y="114.3" size="1.778" layer="95" rot="R180"/>
-<attribute name="VALUE" x="81.28" y="116.84" size="1.778" layer="96" rot="R180"/>
+<instance part="X_1" gate="G$1" x="60.96" y="106.68" smashed="yes"/>
+<instance part="R1" gate="1" x="76.2" y="99.06" smashed="yes" rot="R180">
+<attribute name="NAME" x="73.66" y="104.14" size="1.778" layer="95" rot="R180"/>
+<attribute name="VALUE" x="73.66" y="106.68" size="1.778" layer="96" rot="R180"/>
 </instance>
-<instance part="X_2" gate="G$1" x="91.44" y="106.68" smashed="yes"/>
-<instance part="R2" gate="1" x="86.36" y="78.74" smashed="yes" rot="R180">
-<attribute name="NAME" x="83.82" y="83.82" size="1.778" layer="95" rot="R180"/>
-<attribute name="VALUE" x="83.82" y="86.36" size="1.778" layer="96" rot="R180"/>
+<instance part="X_2" gate="G$1" x="83.82" y="96.52" smashed="yes"/>
+<instance part="R2" gate="1" x="76.2" y="68.58" smashed="yes" rot="R180">
+<attribute name="NAME" x="73.66" y="73.66" size="1.778" layer="95" rot="R180"/>
+<attribute name="VALUE" x="73.66" y="76.2" size="1.778" layer="96" rot="R180"/>
 </instance>
-<instance part="X_3" gate="G$1" x="96.52" y="76.2" smashed="yes"/>
-<instance part="X_4" gate="G$1" x="73.66" y="86.36" smashed="yes"/>
-<instance part="R3" gate="G$1" x="68.58" y="124.46" smashed="yes">
-<attribute name="NAME" x="64.77" y="125.9586" size="1.778" layer="95"/>
-<attribute name="VALUE" x="64.77" y="121.158" size="1.778" layer="96"/>
+<instance part="X_3" gate="G$1" x="86.36" y="66.04" smashed="yes"/>
+<instance part="X_4" gate="G$1" x="63.5" y="76.2" smashed="yes"/>
+<instance part="R3" gate="G$1" x="55.88" y="114.3" smashed="yes">
+<attribute name="NAME" x="52.07" y="115.7986" size="1.778" layer="95"/>
+<attribute name="VALUE" x="52.07" y="110.998" size="1.778" layer="96"/>
 </instance>
-<instance part="R4" gate="G$1" x="68.58" y="93.98" smashed="yes">
-<attribute name="NAME" x="64.77" y="95.4786" size="1.778" layer="95"/>
-<attribute name="VALUE" x="64.77" y="90.678" size="1.778" layer="96"/>
+<instance part="R4" gate="G$1" x="58.42" y="83.82" smashed="yes">
+<attribute name="NAME" x="54.61" y="85.3186" size="1.778" layer="95"/>
+<attribute name="VALUE" x="54.61" y="80.518" size="1.778" layer="96"/>
 </instance>
-<instance part="C1" gate="G$1" x="73.66" y="91.44" smashed="yes">
-<attribute name="NAME" x="75.184" y="91.821" size="1.778" layer="95"/>
-<attribute name="VALUE" x="75.184" y="86.741" size="1.778" layer="96"/>
+<instance part="C1" gate="G$1" x="63.5" y="81.28" smashed="yes">
+<attribute name="NAME" x="65.024" y="81.661" size="1.778" layer="95"/>
+<attribute name="VALUE" x="65.024" y="76.581" size="1.778" layer="96"/>
 </instance>
-<instance part="C2" gate="G$1" x="73.66" y="121.92" smashed="yes">
-<attribute name="NAME" x="75.184" y="122.301" size="1.778" layer="95"/>
-<attribute name="VALUE" x="75.184" y="117.221" size="1.778" layer="96"/>
+<instance part="C2" gate="G$1" x="60.96" y="111.76" smashed="yes">
+<attribute name="NAME" x="62.484" y="112.141" size="1.778" layer="95"/>
+<attribute name="VALUE" x="62.484" y="107.061" size="1.778" layer="96"/>
 </instance>
-<instance part="IC3" gate="A" x="91.44" y="121.92" smashed="yes">
-<attribute name="NAME" x="93.98" y="125.095" size="1.778" layer="95"/>
-<attribute name="VALUE" x="93.98" y="116.84" size="1.778" layer="96"/>
+<instance part="IC3" gate="A" x="83.82" y="111.76" smashed="yes">
+<attribute name="NAME" x="86.36" y="114.935" size="1.778" layer="95"/>
+<attribute name="VALUE" x="86.36" y="106.68" size="1.778" layer="96"/>
 </instance>
-<instance part="IC3" gate="B" x="93.98" y="91.44" smashed="yes">
-<attribute name="NAME" x="96.52" y="94.615" size="1.778" layer="95"/>
-<attribute name="VALUE" x="96.52" y="86.36" size="1.778" layer="96"/>
+<instance part="IC3" gate="B" x="83.82" y="81.28" smashed="yes">
+<attribute name="NAME" x="86.36" y="84.455" size="1.778" layer="95"/>
+<attribute name="VALUE" x="86.36" y="76.2" size="1.778" layer="96"/>
 </instance>
 <instance part="IC3" gate="C" x="38.1" y="137.16" smashed="yes">
@@
 <attribute name="VALUE" x="40.64" y="149.86" size="1.778" layer="96"/>
 </instance>
-<instance part="IC1" gate="A" x="132.08" y="121.92" smashed="yes">
-<attribute name="NAME" x="124.46" y="132.715" size="1.778" layer="95"/>
-<attribute name="VALUE" x="124.46" y="111.76" size="1.778" layer="96"/>
+<instance part="IC1" gate="A" x="119.38" y="111.76" smashed="yes">
+<attribute name="NAME" x="111.76" y="122.555" size="1.778" layer="95"/>
+<attribute name="VALUE" x="111.76" y="101.6" size="1.778" layer="96"/>
 </instance>
-<instance part="IC1" gate="B" x="129.54" y="91.44" smashed="yes">
-<attribute name="NAME" x="121.92" y="102.235" size="1.778" layer="95"/>
-<attribute name="VALUE" x="121.92" y="81.28" size="1.778" layer="96"/>
+<instance part="IC1" gate="B" x="119.38" y="81.28" smashed="yes">
+<attribute name="NAME" x="111.76" y="92.075" size="1.778" layer="95"/>
+<attribute name="VALUE" x="111.76" y="71.12" size="1.778" layer="96"/>
 </instance>
 </instances>
@@
 <net name="N$1" class="0">
 <segment>
-<wire x1="73.66" y1="124.46" x2="83.82" y2="124.46" width="0.1524" layer="91"/>
+<wire x1="60.96" y1="114.3" x2="76.2" y2="114.3" width="0.1524" layer="91"/>
 <pinref part="R3" gate="G$1" pin="2"/>
 <pinref part="C2" gate="G$1" pin="1"/>
-<junction x="73.66" y="124.46"/>
+<junction x="60.96" y="114.3"/>
 <pinref part="IC3" gate="A" pin="+IN"/>
 <pinref part="IC1" gate="A" pin="D"/>
-<wire x1="119.38" y1="124.46" x2="109.22" y2="124.46" width="0.1524" layer="91"/>
-<wire x1="109.22" y1="124.46" x2="109.22" y2="129.54" width="0.1524" layer="91"/>
-<wire x1="109.22" y1="129.54" x2="73.66" y2="129.54" width="0.1524" layer="91"/>
-<wire x1="73.66" y1="129.54" x2="73.66" y2="124.46" width="0.1524" layer="91"/>
+<wire x1="106.68" y1="114.3" x2="96.52" y2="114.3" width="0.1524" layer="91"/>
+<wire x1="96.52" y1="114.3" x2="96.52" y2="119.38" width="0.1524" layer="91"/>
+<wire x1="96.52" y1="119.38" x2="60.96" y2="119.38" width="0.1524" layer="91"/>
+<wire x1="60.96" y1="119.38" x2="60.96" y2="114.3" width="0.1524" layer="91"/>
 </segment>
 </net>
@@
 <pinref part="X_2" gate="G$1" pin="0"/>
 <pinref part="R1" gate="1" pin="1"/>
-<wire x1="91.44" y1="106.68" x2="91.44" y2="109.22" width="0.1524" layer="91"/>
-<wire x1="91.44" y1="109.22" x2="88.9" y2="109.22" width="0.1524" layer="91"/>
+<wire x1="83.82" y1="96.52" x2="83.82" y2="99.06" width="0.1524" layer="91"/>
+<wire x1="83.82" y1="99.06" x2="81.28" y2="99.06" width="0.1524" layer="91"/>
 </segment>
 <segment>
 <pinref part="R2" gate="1" pin="1"/>
 <pinref part="X_3" gate="G$1" pin="0"/>
-<wire x1="91.44" y1="78.74" x2="96.52" y2="78.74" width="0.1524" layer="91"/>
-<wire x1="96.52" y1="78.74" x2="96.52" y2="76.2" width="0.1524" layer="91"/>
+<wire x1="81.28" y1="68.58" x2="86.36" y2="68.58" width="0.1524" layer="91"/>
+<wire x1="86.36" y1="68.58" x2="86.36" y2="66.04" width="0.1524" layer="91"/>
 </segment>
 <segment>
@@
 <segment>
 <pinref part="R1" gate="1" pin="3"/>
-<wire x1="83.82" y1="119.38" x2="83.82" y2="114.3" width="0.1524" layer="91"/>
+<wire x1="76.2" y1="109.22" x2="76.2" y2="104.14" width="0.1524" layer="91"/>
 <pinref part="IC3" gate="A" pin="-IN"/>
 </segment>
@@
 <net name="N$3" class="0">
 <segment>
-<wire x1="73.66" y1="93.98" x2="86.36" y2="93.98" width="0.1524" layer="91"/>
+<wire x1="63.5" y1="83.82" x2="76.2" y2="83.82" width="0.1524" layer="91"/>
 <pinref part="R4" gate="G$1" pin="2"/>
 <pinref part="C1" gate="G$1" pin="1"/>
-<junction x="73.66" y="93.98"/>
+<junction x="63.5" y="83.82"/>
 <pinref part="IC3" gate="B" pin="+IN"/>
-<wire x1="73.66" y1="93.98" x2="73.66" y2="99.06" width="0.1524" layer="91"/>
-<wire x1="73.66" y1="99.06" x2="106.68" y2="99.06" width="0.1524" layer="91"/>
-<wire x1="106.68" y1="99.06" x2="106.68" y2="93.98" width="0.1524" layer="91"/>
+<wire x1="63.5" y1="83.82" x2="63.5" y2="88.9" width="0.1524" layer="91"/>
+<wire x1="63.5" y1="88.9" x2="96.52" y2="88.9" width="0.1524" layer="91"/>
+<wire x1="96.52" y1="88.9" x2="96.52" y2="83.82" width="0.1524" layer="91"/>
 <pinref part="IC1" gate="B" pin="D"/>
-<wire x1="106.68" y1="93.98" x2="116.84" y2="93.98" width="0.1524" layer="91"/>
+<wire x1="96.52" y1="83.82" x2="106.68" y2="83.82" width="0.1524" layer="91"/>
 </segment>
 </net>
@@
 <segment>
 <pinref part="R2" gate="1" pin="3"/>
-<wire x1="86.36" y1="88.9" x2="86.36" y2="83.82" width="0.1524" layer="91"/>
+<wire x1="76.2" y1="78.74" x2="76.2" y2="73.66" width="0.1524" layer="91"/>
 <pinref part="IC3" gate="B" pin="-IN"/>
 </segment>
@@
 <segment>
 <pinref part="IC1" gate="B" pin="CLK"/>
-<wire x1="101.6" y1="91.44" x2="116.84" y2="91.44" width="0.1524" layer="91"/>
+<wire x1="91.44" y1="81.28" x2="106.68" y2="81.28" width="0.1524" layer="91"/>
 <pinref part="IC3" gate="B" pin="OUT"/>
 </segment>
@@
 <pinref part="IC3" gate="A" pin="OUT"/>
 <pinref part="IC1" gate="A" pin="CLK"/>
-<wire x1="99.06" y1="121.92" x2="119.38" y2="121.92" width="0.1524" layer="91"/>
+<wire x1="91.44" y1="111.76" x2="106.68" y2="111.76" width="0.1524" layer="91"/>
 </segment>
 </net>

Commit message: BSPD
Parts:
- added C3, C4: 100uF, rcl:C-EU025-025X050
- added D1: 1N5817-B, diode:1N5817-B
- added IC2: 74ALS805N, 74xx-eu:74ALS805N
- added IC4: LM2576T, v-reg-3:LM2576T
- added IC5: 4013N, 40xx:4013N
- added J1: 22-05-7058-05, con-molex:22-05-7058-05
- added K1: 35701331, relay:35701331
- added L1: 100uH, wurth_elektronik_passive_rev16d:WE-TI_8012
- added R5, R6: (no value), rcl:POTENTIOMETER_PT-10
- C1: value (none) -> 100mF
- C2: value (none) -> 500uF
- R3, R4: value (none) -> 3k
Connections:
- new net 5V: C3.2, IC1P.VDD, IC2P.VCC, IC3P.V+, IC4.FB, IC5P.VDD, L1.2, R1.2, R2.2, R5.2, R6.2
- new net BP: IC3C.+IN, J1-3.S
- new net N$10: IC2B.O, IC5B.CLK
- new net N$11: IC2C.O, R4.1
- new net N$12: IC5B.Q, K11.5
- new net N$13: IC3D.-IN, R6.3
- new net N$14: IC3C.-IN, R5.3
- new net N$15: IC2E.I0, IC2E.I1, IC3C.OUT
- new net N$16: D1.C, IC4.OUT, L1.1
- new net N$17: IC2D.O, IC2F.I0
- new net N$18: IC2E.O, IC2F.I1
- new net N$19: IC2A.O, IC2B.I0, IC2B.I1
- new net N$7: IC2D.I0, IC2D.I1, IC3D.OUT
- new net N$8: IC1B.Q, IC2A.I1
- new net N$9: IC1A.Q, IC2A.I0, IC5B.D
- new net OUT: J1-4.S, K12.S
- new net TPS: IC3D.+IN, J1-2.S
- new net TPS&BP: IC2C.I0, IC2C.I1, IC2F.O, R3.1
- new net VBAT: C4.2, IC4.VIN, J1-1.S, K12.P
- net 0: now also C3.1, C4.1, D1.A, IC1A.R, IC1A.S, IC1B.R, IC1B.S, IC1P.VSS, IC2P.GND, IC3P.V-, IC4.GND, IC4.OFF, IC5B.R, IC5B.S, IC5P.VSS, J1-5.S, K11.3, R5.1, R6.1
Other:
- note added: "Alimentations"
- note added: "Comparateurs"
- note added: "Connecteurs"
- note added: "Logique"
- moved on the sheet: C1, C2, IC1A, IC1B, IC3A, IC3B, IC3C, IC3D, R1, R2, R3, R4

Commit message: de l'élec
Parts:
- added IC7: 4001N, 40xx:4001N
- IC2: value 74ALS805N -> 4001N; device 74xx-eu:74ALS805N -> 40xx:4001N
- J1: value 22-05-7058-05 -> 22-05-7068-06; device con-molex:22-05-7058-05 -> con-molex:22-05-7068-06
Connections:
- new net N$21: IC1A.R, IC7C.O
- new net SDC: J1-5.S, K12.P
- net 0: now also IC2P.VSS, IC7P.VSS, J1-6.S; no longer IC1A.R, IC2P.GND, J1-5.S
- net 5V: now also IC2P.VDD, IC7P.VDD; no longer IC2P.VCC
- net N$11: now also IC7B.O; no longer IC2C.O
- net N$15: now also IC2C.I0, IC2C.I1; no longer IC2E.I0, IC2E.I1
- net N$17: now also IC7A.I0; no longer IC2F.I0
- net N$18: now also IC2C.O, IC7A.I1; no longer IC2E.O, IC2F.I1
- net N$8: now also IC7C.I0, IC7C.I1
- net TPS&BP: now also IC7A.O, IC7B.I0, IC7B.I1; no longer IC2C.I0, IC2C.I1, IC2F.O
- net VBAT: no longer K12.P
Other:
- moved on the sheet: C1, IC1B, IC2C, IC3B, R2, R4

Commit message: élec
Parts:
- removed R1, R2, R5, R6: (no value), rcl:POTENTIOMETER_PT-10
- added R10, R7, R8, R9: (no value), rcl:POTENTIOMETER_PT_SPIN
Connections:
- net SDC renamed SDS
- net 0: now also R10.1, R7.1, R8.1, R9.1; no longer R1.1, R2.1, R5.1, R6.1
- net 5V: now also R10.2, R7.2, R8.2, R9.2; no longer R1.2, R2.2, R5.2, R6.2
- net N$13: now also R10.3; no longer R6.3
- net N$14: now also R8.3; no longer R5.3
- net N$2: now also R7.3; no longer R1.3
- net N$4: now also R9.3; no longer R2.3
Other:
- moved on the sheet: J1-1, J1-2, J1-3, J1-4, J1-5, J1-6

Commit message: BSPD
Parts:
- removed IC1: 4013N, 40xx:4013N
- removed IC3: LM2901N, linear:LM2901N
- removed R3, R4: 3k, rcl:R-EU_0204/7
- removed R7, R9: (no value), rcl:POTENTIOMETER_PT_SPIN
- added C5, C6: 0.01uF, rcl:C-EU025-025X050
- added IC6, IC8: NE555, st-microelectronics:NE555
- added IC9: LM393N, linear:LM393N
- added R1, R2: (no value), rcl:R-EU_0207/10
- C1: value 100mF -> 0.01uF
- C2: value 500uF -> 0.01uF
Connections:
- removed net N$21: IC1A.R, IC7C.O
- net 0: now also C1.1, C2.1, C5.1, C6.1, IC6.GND, IC8.GND, IC9P.V-; no longer C1.2, C2.2, IC1A.S, IC1B.R, IC1B.S, IC1P.VSS, IC3P.V-, R7.1, R9.1
- net 5V: now also IC6.VCC+, IC8.VCC+, IC9P.V+, R1.2, R2.2; no longer IC1P.VDD, IC3P.V+, R7.2, R9.2
- net BP: now also IC9B.+IN; no longer IC3C.+IN
- net N$1: now also C1.2, IC8.CON; no longer C2.1, IC1A.D, IC3A.+IN, R3.2
- net N$11: now also IC6.OUT, IC7D.I1; no longer IC7B.O, R4.1
- net N$13: now also IC9A.-IN; no longer IC3D.-IN
- net N$14: now also IC9B.-IN; no longer IC3C.-IN
- net N$15: now also IC9B.OUT; no longer IC3C.OUT
- net N$2: now also IC7B.O, IC7C.I0, IC8./RES, IC8.TRI; no longer IC3A.-IN, R7.3
- net N$3: now also C2.2, IC8.DIS, IC8.TRE, R1.1; no longer C1.1, IC1B.D, IC3B.+IN, R4.2
- net N$4: now also IC7C.I1, IC8.OUT; no longer IC3B.-IN, R9.3
- net N$5: now also C6.2, IC6.DIS, IC6.TRE, R2.1; no longer IC1B.CLK, IC3B.OUT
- net N$6: now also C5.2, IC6.CON; no longer IC1A.CLK, IC3A.OUT
- net N$7: now also IC9A.OUT; no longer IC3D.OUT
- net N$8: now also IC7C.O; no longer IC1B.Q, IC7C.I0, IC7C.I1
- net N$9: now also IC7D.O; no longer IC1A.Q
- net TPS: now also IC9A.+IN; no longer IC3D.+IN
- net TPS&BP: now also IC6./RES, IC6.TRI, IC7D.I0; no longer R3.1
Other:
- moved on the sheet: C1, C2, IC7B, IC7C, IC7P
