File: EL - Electrical/Autre/Tableau de bord/Carte élecs/Afficheur temp/rapport.sch (EAGLE design)
At the start: 25 parts, among them IC1 MCP23008P, IC2 MCP23008P, X1 22-23-2041

Commit message: afficheur temp
Connections:
- net GP10: no longer R1A.2
- net GP11: no longer R1B.2
- net GP13: no longer R1F.2, R2D.2
- net GP15: no longer R2A.2
- net GP16: now also R2D.2
- net GP17: now also R2E.2
- net GP20: now also R3AB.2; no longer R2B.2
- net GP21: now also R2F.2
- net GP22: now also R2G.2
- net GP23: now also R2A.2; no longer R2E.2
- net GP24: now also R2B.2; no longer R2F.2
- net GP25: now also R1F.2; no longer R2G.2
- net GP26: now also R1A.2
- net GP27: now also R1B.2; no longer R3AB.2
- net SCL: now also C2.1, R1.1, X1-3.S; no longer C3.1, R2.2, X1-2.S
- net SDA: now also C3.1, R2.2, X1-2.S; no longer C2.1, R1.1, X1-3.S

Commit message: Changement afficheur temp
Connections:
- net GP10: now also R2B.2; no longer R1C.2
- net GP11: now also R2A.2; no longer R1G.2
- net GP12: now also R2F.2; no longer R1D.2
- net GP13: now also R2G.2; no longer R1E.2
- net GP20: now also R1G.2; no longer R3AB.2
- net GP21: now also R1C.2; no longer R2F.2
- net GP22: now also R1D.2; no longer R2G.2
- net GP23: now also R1E.2; no longer R2A.2
- net GP24: now also R1F.2; no longer R2B.2
- net GP25: now also R1A.2; no longer R1F.2
- net GP26: now also R1B.2; no longer R1A.2
- net GP27: now also R3AB.2; no longer R1B.2
Changed lines of the file:
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@@
 </segment>
 <segment>
-<pinref part="R1E" gate="G$1" pin="2"/>
-<wire x1="45.72" y1="142.24" x2="40.64" y2="142.24" width="0.1524" layer="91"/>
-<label x="40.64" y="142.24" size="1.778" layer="95" rot="R180" xref="yes"/>
+<pinref part="R2G" gate="G$1" pin="2"/>
+<wire x1="45.72" y1="109.22" x2="43.18" y2="109.22" width="0.1524" layer="91"/>
+<label x="43.18" y="109.22" size="1.778" layer="95" rot="R180" xref="yes"/>
 </segment>
 </net>
@@
 </segment>
 <segment>
-<pinref part="R1D" gate="G$1" pin="2"/>
-<wire x1="45.72" y1="144.78" x2="31.75" y2="144.78" width="0.1524" layer="91"/>
-<label x="31.75" y="144.78" size="1.778" layer="95" rot="R180" xref="yes"/>
+<pinref part="R2F" gate="G$1" pin="2"/>
+<wire x1="45.72" y1="111.76" x2="34.29" y2="111.76" width="0.1524" layer="91"/>
+<label x="34.29" y="111.76" size="1.778" layer="95" rot="R180" xref="yes"/>
 </segment>
 </net>
@@
 </segment>
 <segment>
-<pinref part="R1G" gate="G$1" pin="2"/>
-<wire x1="45.72" y1="137.16" x2="40.64" y2="137.16" width="0.1524" layer="91"/>
-<label x="40.64" y="137.16" size="1.778" layer="95" rot="R180" xref="yes"/>
+<pinref part="R2A" gate="G$1" pin="2"/>
+<wire x1="45.72" y1="124.46" x2="43.18" y2="124.46" width="0.1524" layer="91"/>
+<label x="43.18" y="124.46" size="1.778" layer="95" rot="R180" xref="yes"/>
 </segment>
 </net>
@@
 </segment>
 <segment>
-<pinref part="R1C" gate="G$1" pin="2"/>
-<wire x1="45.72" y1="147.32" x2="40.64" y2="147.32" width="0.1524" layer="91"/>
-<label x="40.64" y="147.32" size="1.778" layer="95" rot="R180" xref="yes"/>
+<pinref part="R2B" gate="G$1" pin="2"/>
+<wire x1="45.72" y1="121.92" x2="34.29" y2="121.92" width="0.1524" layer="91"/>
+<label x="34.29" y="121.92" size="1.778" layer="95" rot="R180" xref="yes"/>
 </segment>
 </net>
@@
 </segment>
 <segment>
-<pinref part="R1B" gate="G$1" pin="2"/>
-<wire x1="45.72" y1="149.86" x2="31.75" y2="149.86" width="0.1524" layer="91"/>
-<label x="31.75" y="149.86" size="1.778" layer="95" rot="R180" xref="yes"/>
+<pinref part="R3AB" gate="G$1" pin="2"/>
+<wire x1="95.25" y1="152.4" x2="93.98" y2="152.4" width="0.1524" layer="91"/>
+<label x="93.98" y="148.59" size="1.778" layer="95" rot="R180" xref="yes"/>
+<wire x1="93.98" y1="152.4" x2="93.98" y2="148.59" width="0.1524" layer="91"/>
 </segment>
 </net>
@@
 </segment>
 <segment>
-<pinref part="R1A" gate="G$1" pin="2"/>
-<wire x1="45.72" y1="152.4" x2="40.64" y2="152.4" width="0.1524" layer="91"/>
-<label x="40.64" y="152.4" size="1.778" layer="95" rot="R180" xref="yes"/>
+<pinref part="R1B" gate="G$1" pin="2"/>
+<wire x1="45.72" y1="149.86" x2="31.75" y2="149.86" width="0.1524" layer="91"/>
+<label x="31.75" y="149.86" size="1.778" layer="95" rot="R180" xref="yes"/>
 </segment>
 </net>
@@
 </segment>
 <segment>
-<pinref part="R1F" gate="G$1" pin="2"/>
-<wire x1="45.72" y1="139.7" x2="31.75" y2="139.7" width="0.1524" layer="91"/>
-<label x="31.75" y="139.7" size="1.778" layer="95" rot="R180" xref="yes"/>
+<pinref part="R1A" gate="G$1" pin="2"/>
+<wire x1="45.72" y1="152.4" x2="40.64" y2="152.4" width="0.1524" layer="91"/>
+<label x="40.64" y="152.4" size="1.778" layer="95" rot="R180" xref="yes"/>
 </segment>
 </net>
@@
 </segment>
 <segment>
-<pinref part="R2B" gate="G$1" pin="2"/>
-<wire x1="45.72" y1="121.92" x2="34.29" y2="121.92" width="0.1524" layer="91"/>
-<label x="34.29" y="121.92" size="1.778" layer="95" rot="R180" xref="yes"/>
+<pinref part="R1F" gate="G$1" pin="2"/>
+<wire x1="45.72" y1="139.7" x2="31.75" y2="139.7" width="0.1524" layer="91"/>
+<label x="31.75" y="139.7" size="1.778" layer="95" rot="R180" xref="yes"/>
 </segment>
 </net>
@@
 </segment>
 <segment>
-<pinref part="R2A" gate="G$1" pin="2"/>
-<wire x1="45.72" y1="124.46" x2="43.18" y2="124.46" width="0.1524" layer="91"/>
-<label x="43.18" y="124.46" size="1.778" layer="95" rot="R180" xref="yes"/>
+<pinref part="R1E" gate="G$1" pin="2"/>
+<wire x1="45.72" y1="142.24" x2="40.64" y2="142.24" width="0.1524" layer="91"/>
+<label x="40.64" y="142.24" size="1.778" layer="95" rot="R180" xref="yes"/>
 </segment>
 </net>
@@
 </segment>
 <segment>
-<pinref part="R2G" gate="G$1" pin="2"/>
-<wire x1="45.72" y1="109.22" x2="43.18" y2="109.22" width="0.1524" layer="91"/>
-<label x="43.18" y="109.22" size="1.778" layer="95" rot="R180" xref="yes"/>
+<pinref part="R1D" gate="G$1" pin="2"/>
+<wire x1="45.72" y1="144.78" x2="31.75" y2="144.78" width="0.1524" layer="91"/>
+<label x="31.75" y="144.78" size="1.778" layer="95" rot="R180" xref="yes"/>
 </segment>
 </net>
@@
 </segment>
 <segment>
-<pinref part="R2F" gate="G$1" pin="2"/>
-<wire x1="45.72" y1="111.76" x2="34.29" y2="111.76" width="0.1524" layer="91"/>
-<label x="34.29" y="111.76" size="1.778" layer="95" rot="R180" xref="yes"/>
+<pinref part="R1C" gate="G$1" pin="2"/>
+<wire x1="45.72" y1="147.32" x2="40.64" y2="147.32" width="0.1524" layer="91"/>
+<label x="40.64" y="147.32" size="1.778" layer="95" rot="R180" xref="yes"/>
 </segment>
 </net>
@@
 </segment>
 <segment>
-<pinref part="R3AB" gate="G$1" pin="2"/>
-<wire x1="95.25" y1="152.4" x2="93.98" y2="152.4" width="0.1524" layer="91"/>
-<label x="93.98" y="148.59" size="1.778" layer="95" rot="R180" xref="yes"/>
-<wire x1="93.98" y1="152.4" x2="93.98" y2="148.59" width="0.1524" layer="91"/>
+<pinref part="R1G" gate="G$1" pin="2"/>
+<wire x1="45.72" y1="137.16" x2="40.64" y2="137.16" width="0.1524" layer="91"/>
+<label x="40.64" y="137.16" size="1.778" layer="95" rot="R180" xref="yes"/>
 </segment>
 </net>
