File: EL - Electrical/Autre/Tableau de bord/Carte élecs/Afficheur temp/Temp.sch (EAGLE design)
At the start: 26 parts, among them IC1 MCP23008P, IC2 MCP23008P, X1 22-23-2041

Commit message: afficheur tdb
Other:
- note added: "Afficheur Temp v1.4"
- note removed: "Afficheur Temp v1.0"
Changed lines of the file:
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@@
 <part name="P+5" library="supply1" library_urn="urn:adsk.eagle:library:371" deviceset="+5V" device=""/>
 <part name="R1A" library="rcl" library_urn="urn:adsk.eagle:library:334" deviceset="R-EU_" device="0204/7" package3d_urn="urn:adsk.eagle:package:23498/1" value="470"/>
-<part name="FRAME1" library="frames" library_urn="urn:adsk.eagle:library:229" deviceset="A4L-LOC" device=""/>
+<part name="FRAME1" library="frames" library_urn="urn:adsk.eagle:library:229" deviceset="A4L-LOC" device="" value="Temp display"/>
 <part name="LED2" library="display-kingbright" library_urn="urn:adsk.eagle:library:213" deviceset="B?56-11*WA" device="A" package3d_urn="urn:adsk.eagle:package:13080/1" technology="E"/>
 <part name="R1B" library="rcl" library_urn="urn:adsk.eagle:library:334" deviceset="R-EU_" device="0204/7" package3d_urn="urn:adsk.eagle:package:23498/1" value="470"/>
@@
 <plain>
 <text x="167.14" y="9.16" size="5.08" layer="94">Afficheur
-Temp v1.0</text>
+Temp v1.4</text>
 <text x="216.44" y="20.32" size="2.54" layer="94">EPSA Saison 2018/2019</text>
 <wire x1="180.8" y1="166.26" x2="180.8" y2="95.14" width="0.1524" layer="97"/>

Commit message: plein de choses
Parts:
- removed C2: 135pF, rcl:C-EU025-025X050
- removed C3: 135 pF, rcl:C-EU025-025X050
Connections:
- net GND: no longer C2.2, C3.2
- net SCL: no longer C2.1
- net SDA: no longer C3.1
Changed lines of the file:
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@@
 <part name="P+1" library="supply1" library_urn="urn:adsk.eagle:library:371" deviceset="+5V" device=""/>
 <part name="C1" library="rcl" library_urn="urn:adsk.eagle:library:334" deviceset="C-EU" device="025-025X050" package3d_urn="urn:adsk.eagle:package:23629/2" value="500pF"/>
-<part name="C2" library="rcl" library_urn="urn:adsk.eagle:library:334" deviceset="C-EU" device="025-025X050" package3d_urn="urn:adsk.eagle:package:23629/2" value="135pF"/>
-<part name="GND4" library="supply1" library_urn="urn:adsk.eagle:library:371" deviceset="GND" device=""/>
-<part name="C3" library="rcl" library_urn="urn:adsk.eagle:library:334" deviceset="C-EU" device="025-025X050" package3d_urn="urn:adsk.eagle:package:23629/2" value="135 pF"/>
-<part name="GND5" library="supply1" library_urn="urn:adsk.eagle:library:371" deviceset="GND" device=""/>
 <part name="P+4" library="supply1" library_urn="urn:adsk.eagle:library:371" deviceset="+5V" device=""/>
 <part name="P+6" library="supply1" library_urn="urn:adsk.eagle:library:371" deviceset="+5V" device=""/>
@@
 <attribute name="VALUE" x="201.104" y="51.631" size="1.778" layer="96"/>
 </instance>
-<instance part="C2" gate="G$1" x="208.74" y="140.86" smashed="yes">
-<attribute name="NAME" x="210.264" y="141.241" size="1.778" layer="95"/>
-<attribute name="VALUE" x="210.264" y="136.161" size="1.778" layer="96"/>
-</instance>
-<instance part="GND4" gate="1" x="208.74" y="133.24" smashed="yes">
-<attribute name="VALUE" x="206.2" y="130.7" size="1.778" layer="96"/>
-</instance>
-<instance part="C3" gate="G$1" x="208.74" y="112.92" smashed="yes">
-<attribute name="NAME" x="210.264" y="113.301" size="1.778" layer="95"/>
-<attribute name="VALUE" x="210.264" y="108.221" size="1.778" layer="96"/>
-</instance>
-<instance part="GND5" gate="1" x="208.74" y="105.3" smashed="yes">
-<attribute name="VALUE" x="206.2" y="102.76" size="1.778" layer="96"/>
-</instance>
 <instance part="P+4" gate="1" x="208.74" y="156.1" smashed="yes">
 <attribute name="VALUE" x="206.2" y="151.02" size="1.778" layer="96" rot="R90"/>
@@
 <wire x1="199.58" y1="51.25" x2="188.104" y2="51.25" width="0.1524" layer="91"/>
 <junction x="199.58" y="51.25"/>
-</segment>
-<segment>
-<pinref part="GND4" gate="1" pin="GND"/>
-<pinref part="C2" gate="G$1" pin="2"/>
-</segment>
-<segment>
-<pinref part="C3" gate="G$1" pin="2"/>
-<pinref part="GND5" gate="1" pin="GND"/>
 </segment>
 <segment>
@@
 </segment>
 <segment>
-<pinref part="C2" gate="G$1" pin="1"/>
 <junction x="208.74" y="143.4"/>
 <pinref part="R1" gate="G$1" pin="1"/>
@@
 <wire x1="208.74" y1="115.46" x2="221.44" y2="115.46" width="0.1524" layer="91"/>
 <pinref part="R2" gate="G$1" pin="2"/>
-<pinref part="C3" gate="G$1" pin="1"/>
 <junction x="208.74" y="115.46"/>
 <label x="221.44" y="115.46" size="1.778" layer="95" xref="yes"/>
