File: EL - Electrical/Autre/Tableau de bord/Carte élecs/Afficheur temp/TEMP.BRD (EAGLE design)
At the start: 79 x 42 mm, 25 parts, among them IC1 MCP23008P, IC2 MCP23008P, X1 22-23-2041

Commit message: MAJ plan afficheur temp
Parts:
- moved R2 62.5 mm to (65.7, 7.62)
- moved IC1 55.3 mm to (76.8, 21.9), turned to 90 degrees
- moved C2 49.0 mm to (50.8, 10.2), turned to 0 degrees
- moved C3 48.0 mm to (53.3, 5.08)
- moved X1 44.6 mm to (41.9, 5.08), turned to 0 degrees
- moved R2DP 37.6 mm to (19.1, 28.9), turned to 0 degrees
- moved R1E 30.5 mm to (19.1, 18.7), turned to 180 degrees
- moved R1F 27.9 mm to (19.1, 21.3), turned to 180 degrees
- moved C1 27.3 mm to (33.7, 4.76), turned to 90 degrees
- moved R1D 27.2 mm to (19.1, 16.2), turned to 180 degrees
- moved R1A 24.4 mm to (19.1, 23.8), turned to 180 degrees
- moved R1G 23.5 mm to (19.1, 11.1), turned to 180 degrees
- moved R1C 21.6 mm to (19.1, 13.7), turned to 180 degrees
- moved R1B 20.9 mm to (19.1, 26.4), turned to 180 degrees
- moved R2G 19.1 mm to (66.4, 21.9), turned to 0 degrees
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Connections:
- net GP10: now also R2B.2; no longer R1C.2
- net GP11: now also R2A.2; no longer R1G.2
- net GP12: now also R3AB.2; no longer R1D.2
- net GP13: now also R2F.2; no longer R1E.2
- net GP14: now also R2G.2; no longer R2DP.1
- net GP20: now also R1G.2; no longer R3AB.2
- net GP21: now also R1C.2; no longer R2F.2
- net GP22: now also R1D.2; no longer R2G.2
- net GP23: now also R1E.2; no longer R2A.2
- net GP24: now also R1F.2; no longer R2B.2
- net GP25: now also R1A.2; no longer R1F.2
- net GP26: now also R1B.2; no longer R1A.2
- net GP27: now also R2DP.1; no longer R1B.2
Routing:
- net GND: track 63.2 -> 129.5 mm
- net SCL: track 45.6 -> 101.1 mm
- net SDA: track 52.5 -> 101.3 mm
- net GP20: track 33.9 -> 2.22 mm
- net GP12: track 31.4 -> 0.00 mm
- net GP14: track 31.4 -> 0.00 mm
- net GP13: track 31.4 -> 0.00 mm
- net GP23: track 31.4 -> 2.22 mm
- net GP22: track 31.4 -> 2.22 mm
- net GP21: track 31.4 -> 2.22 mm
- net GP24: track 31.4 -> 2.22 mm
- net GP17: track 31.4 -> 2.86 mm
- net GP16: track 31.4 -> 2.86 mm
- net GP15: track 31.4 -> 2.86 mm
- net GP11: track 31.4 -> 2.86 mm
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- removed copper zone on layer 1, net +5V
- removed copper zone on layer 16, net GND
Other:
- board size 79 x 42 mm -> 82 x 38 mm

Commit message: changement d'adresse afficheur temp
Connections:
- net +5V: now also IC1.4, IC2.5; no longer IC1.5, IC2.4
- net GND: now also IC1.5, IC2.4; no longer IC1.4, IC2.5
Routing:
- net +5V: track 144.7 -> 143.4 mm
- net GND: track 129.5 -> 130.7 mm
Changed lines of the file:
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@@
 <contactref element="X1" pad="4"/>
 <contactref element="IC1" pad="3"/>
-<contactref element="IC1" pad="4"/>
 <contactref element="IC1" pad="9"/>
 <contactref element="IC2" pad="9"/>
-<contactref element="IC2" pad="5"/>
 <contactref element="IC2" pad="3"/>
 <wire x1="5.3975" y1="11.1125" x2="10.4775" y2="6.0325" width="0.1524" layer="16"/>
 <wire x1="10.4775" y1="6.0325" x2="33.655" y2="6.0325" width="0.1524" layer="16"/>
-<wire x1="7.62" y1="19.05" x2="7.62" y2="13.335" width="0.1524" layer="16"/>
-<wire x1="5.3975" y1="11.1125" x2="7.62" y2="13.335" width="0.1524" layer="16"/>
-<wire x1="7.62" y1="19.05" x2="5.3975" y2="21.2725" width="0.1524" layer="16"/>
+<wire x1="7.62" y1="13.335" x2="5.3975" y2="11.1125" width="0.1524" layer="16"/>
 <wire x1="45.72" y1="5.08" x2="45.87875" y2="4.92125" width="0.1524" layer="16"/>
 <wire x1="45.87875" y1="4.92125" x2="46.99" y2="3.81" width="0.1524" layer="16"/>
@@
 <wire x1="61.2775" y1="8.255" x2="72.0725" y2="8.255" width="0.1524" layer="16"/>
 <wire x1="72.0725" y1="8.255" x2="80.645" y2="16.8275" width="0.1524" layer="16"/>
-<wire x1="80.645" y1="16.8275" x2="80.645" y2="19.3675" width="0.1524" layer="16"/>
-<wire x1="80.645" y1="19.3675" x2="78.105" y2="21.9075" width="0.1524" layer="16"/>
-<wire x1="78.105" y1="21.9075" x2="78.105" y2="29.5275" width="0.1524" layer="16"/>
 <wire x1="33.655" y1="6.0325" x2="37.5191" y2="2.1684" width="0.1524" layer="16"/>
 <wire x1="43.1259" y1="2.1684" x2="45.87875" y2="4.92125" width="0.1524" layer="16"/>
 <wire x1="37.5191" y1="2.1684" x2="43.1259" y2="2.1684" width="0.1524" layer="16"/>
-<wire x1="7.62" y1="24.13" x2="5.3975" y2="26.3525" width="0.1524" layer="16"/>
-<wire x1="5.3975" y1="21.2725" x2="7.62" y2="23.495" width="0.1524" layer="16"/>
-<wire x1="7.62" y1="23.495" x2="7.62" y2="24.13" width="0.1524" layer="16"/>
-<wire x1="80.645" y1="32.0675" x2="78.4225" y2="29.845" width="0.1524" layer="16"/>
-<wire x1="78.4225" y1="29.845" x2="78.105" y2="29.5275" width="0.1524" layer="16"/>
+<contactref element="IC1" pad="5"/>
+<contactref element="IC2" pad="4"/>
+<wire x1="5.3975" y1="26.3525" x2="5.3975" y2="23.8125" width="0.1524" layer="16"/>
+<wire x1="5.3975" y1="23.8125" x2="7.62" y2="21.59" width="0.1524" layer="16"/>
+<wire x1="7.62" y1="21.59" x2="7.62" y2="13.335" width="0.1524" layer="16"/>
+<wire x1="80.645" y1="16.8275" x2="78.105" y2="19.3675" width="0.1524" layer="16"/>
+<wire x1="78.105" y1="19.3675" x2="78.105" y2="20.0025" width="0.1524" layer="16"/>
+<wire x1="78.105" y1="20.0025" x2="80.01" y2="21.9075" width="0.1524" layer="16"/>
+<wire x1="80.01" y1="21.9075" x2="80.645" y2="21.9075" width="0.1524" layer="16"/>
+<wire x1="80.645" y1="21.9075" x2="78.105" y2="24.4475" width="0.1524" layer="16"/>
+<wire x1="78.105" y1="24.4475" x2="78.105" y2="30.48" width="0.1524" layer="16"/>
+<wire x1="78.105" y1="30.48" x2="79.6925" y2="32.0675" width="0.1524" layer="16"/>
+<wire x1="79.6925" y1="32.0675" x2="80.645" y2="32.0675" width="0.1524" layer="16"/>
 </signal>
 <signal name="+5V">
@@
 <contactref element="R1" pad="2"/>
 <contactref element="X1" pad="1"/>
-<contactref element="IC1" pad="5"/>
 <contactref element="IC1" pad="6"/>
 <contactref element="IC1" pad="18"/>
@@
 <contactref element="IC2" pad="6"/>
 <contactref element="IC2" pad="18"/>
-<contactref element="IC2" pad="4"/>
 <contactref element="LED2" pad="19"/>
 <contactref element="LED2" pad="3"/>
@@
 <wire x1="65.7225" y1="11.43" x2="72.7075" y2="11.43" width="0.1524" layer="1"/>
 <wire x1="72.7075" y1="11.43" x2="73.025" y2="11.7475" width="0.1524" layer="1"/>
-<wire x1="73.025" y1="11.7475" x2="77.1525" y2="15.875" width="0.1524" layer="1"/>
-<wire x1="77.1525" y1="15.875" x2="77.1525" y2="20.32" width="0.1524" layer="1"/>
-<wire x1="77.1525" y1="20.32" x2="78.74" y2="21.9075" width="0.1524" layer="1"/>
-<wire x1="78.74" y1="21.9075" x2="80.645" y2="21.9075" width="0.1524" layer="1"/>
 <wire x1="38.1" y1="5.08" x2="35.2425" y2="5.08" width="0.1524" layer="1"/>
 <wire x1="35.2425" y1="5.08" x2="33.655" y2="3.4925" width="0.1524" layer="1"/>
@@
 <wire x1="38.1" y1="5.08" x2="44.45" y2="11.43" width="0.1524" layer="1"/>
 <wire x1="44.45" y1="11.43" x2="57.4675" y2="11.43" width="0.1524" layer="1"/>
-<wire x1="80.645" y1="21.9075" x2="80.645" y2="24.4475" width="0.1524" layer="1"/>
 <wire x1="36.5125" y1="29.845" x2="38.735" y2="27.6225" width="0.1524" layer="1"/>
 <wire x1="33.9725" y1="29.845" x2="36.5125" y2="29.845" width="0.1524" layer="1"/>
 <wire x1="13.0175" y1="31.4325" x2="32.385" y2="31.4325" width="0.1524" layer="16"/>
 <wire x1="32.385" y1="31.4325" x2="33.9725" y2="29.845" width="0.1524" layer="16"/>
-<wire x1="5.3975" y1="23.8125" x2="13.0175" y2="31.4325" width="0.1524" layer="1"/>
-<wire x1="5.3975" y1="18.7325" x2="6.35" y2="18.7325" width="0.1524" layer="1"/>
-<wire x1="6.35" y1="18.7325" x2="7.62" y2="20.0025" width="0.1524" layer="1"/>
-<wire x1="7.62" y1="20.0025" x2="7.62" y2="21.9075" width="0.1524" layer="1"/>
-<wire x1="7.62" y1="21.9075" x2="5.715" y2="23.8125" width="0.1524" layer="1"/>
-<wire x1="5.715" y1="23.8125" x2="5.3975" y2="23.8125" width="0.1524" layer="1"/>
+<contactref element="IC1" pad="4"/>
+<contactref element="IC2" pad="5"/>
+<wire x1="5.3975" y1="18.7325" x2="5.3975" y2="21.2725" width="0.1524" layer="1"/>
+<wire x1="10.8331" y1="26.7081" x2="5.3975" y2="21.2725" width="0.1524" layer="1"/>
+<wire x1="13.0175" y1="31.4325" x2="13.0048625" y2="31.4325" width="0.1524" layer="1"/>
+<wire x1="13.0048625" y1="31.4325" x2="10.8331" y2="29.2607375" width="0.1524" layer="1"/>
+<wire x1="10.8331" y1="29.2607375" x2="10.8331" y2="26.7081" width="0.1524" layer="1"/>
+<wire x1="80.645" y1="19.3675" x2="73.025" y2="11.7475" width="0.1524" layer="1"/>
+<wire x1="80.645" y1="19.3675" x2="78.105" y2="21.9075" width="0.1524" layer="1"/>
+<wire x1="78.105" y1="21.9075" x2="78.105" y2="22.5425" width="0.1524" layer="1"/>
+<wire x1="78.105" y1="22.5425" x2="80.01" y2="24.4475" width="0.1524" layer="1"/>
+<wire x1="80.01" y1="24.4475" x2="80.645" y2="24.4475" width="0.1524" layer="1"/>
 </signal>
 <signal name="SCL">

Commit message: légère modifs à terminer
Parts:
- added R3AB1: 230, rcl:0204/7
- R3AB: value 470 -> 230
- moved R2A 2.54 mm to (66.4, 32.1)
- moved R2B 2.54 mm to (66.4, 34.6)
Connections:
- new net N$16: LED2.24, R3AB1.1
- net GP12: now also R3AB1.2
- net N$17: no longer LED2.24
Routing:
- net N$16: track 0.00 -> 14.8 mm
- net GP12: track 0.00 -> 5.40 mm
- net GP14: track 0.00 -> 2.86 mm
- net GP13: track 0.00 -> 2.86 mm
- net N$17: track 14.5 -> 12.0 mm
- net GP27: track 0.00 -> 2.22 mm
- net GP11: track 2.86 -> 3.91 mm
- net GP10: track 2.86 -> 3.91 mm
- net SCL: track 101.1 -> 101.7 mm
- net N$9: track 24.9 -> 25.5 mm
- added copper zone on layer 16, net GND
Changed lines of the file:
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@@
 <attribute name="VALUE" x="8.3185" y="31.4325" size="1.778" layer="27" ratio="10" rot="R270"/>
 </element>
-<element name="R2A" library="rcl" library_urn="urn:adsk.eagle:library:334" package="0204/7" package3d_urn="urn:adsk.eagle:package:23498/1" value="470" x="66.3575" y="29.5275" smashed="yes">
-<attribute name="NAME" x="60.96" y="27.6479" size="0.9906" layer="25" ratio="10"/>
-<attribute name="SPICEPREFIX" value="R" x="66.3575" y="29.5275" size="1.778" layer="27" display="off"/>
-<attribute name="VALUE" x="64.7319" y="29.0449" size="0.9906" layer="27" ratio="10"/>
-</element>
-<element name="R2B" library="rcl" library_urn="urn:adsk.eagle:library:334" package="0204/7" package3d_urn="urn:adsk.eagle:package:23498/1" value="470" x="66.3575" y="32.0675" smashed="yes">
+<element name="R2A" library="rcl" library_urn="urn:adsk.eagle:library:334" package="0204/7" package3d_urn="urn:adsk.eagle:package:23498/1" value="470" x="66.3575" y="32.0675" smashed="yes">
 <attribute name="NAME" x="60.96" y="30.1879" size="0.9906" layer="25" ratio="10"/>
 <attribute name="SPICEPREFIX" value="R" x="66.3575" y="32.0675" size="1.778" layer="27" display="off"/>
 <attribute name="VALUE" x="64.7319" y="31.5849" size="0.9906" layer="27" ratio="10"/>
+</element>
+<element name="R2B" library="rcl" library_urn="urn:adsk.eagle:library:334" package="0204/7" package3d_urn="urn:adsk.eagle:package:23498/1" value="470" x="66.3575" y="34.6075" smashed="yes">
+<attribute name="NAME" x="60.96" y="32.7279" size="0.9906" layer="25" ratio="10"/>
+<attribute name="SPICEPREFIX" value="R" x="66.3575" y="34.6075" size="1.778" layer="27" display="off"/>
+<attribute name="VALUE" x="64.7319" y="34.1249" size="0.9906" layer="27" ratio="10"/>
 </element>
 <element name="R2C" library="rcl" library_urn="urn:adsk.eagle:library:334" package="0204/7" package3d_urn="urn:adsk.eagle:package:23498/1" value="470" x="66.3575" y="19.3675" smashed="yes">
@@
 <attribute name="VALUE" x="20.6756" y="29.3751" size="0.9906" layer="27" ratio="10" rot="R180"/>
 </element>
-<element name="R3AB" library="rcl" library_urn="urn:adsk.eagle:library:334" package="0204/7" package3d_urn="urn:adsk.eagle:package:23498/1" value="470" x="66.3575" y="26.9875" smashed="yes">
+<element name="R3AB" library="rcl" library_urn="urn:adsk.eagle:library:334" package="0204/7" package3d_urn="urn:adsk.eagle:package:23498/1" value="230" x="66.3575" y="26.9875" smashed="yes">
 <attribute name="NAME" x="60.0075" y="25.1079" size="0.9906" layer="25" ratio="10"/>
 <attribute name="SPICEPREFIX" value="R" x="66.3575" y="26.9875" size="1.778" layer="27" display="off"/>
 <attribute name="VALUE" x="64.7319" y="26.5049" size="0.9906" layer="27" ratio="10"/>
+</element>
+<element name="R3AB1" library="rcl" library_urn="urn:adsk.eagle:library:334" package="0204/7" package3d_urn="urn:adsk.eagle:package:23498/1" value="230" x="66.3575" y="29.5275" smashed="yes">
+<attribute name="NAME" x="59.3725" y="27.6479" size="0.9906" layer="25" ratio="10"/>
+<attribute name="SPICEPREFIX" value="R" x="66.3575" y="29.5275" size="1.778" layer="27" display="off"/>
+<attribute name="VALUE" x="64.7319" y="29.0449" size="0.9906" layer="27" ratio="10"/>
 </element>
 </elements>
@@
 <wire x1="78.105" y1="30.48" x2="79.6925" y2="32.0675" width="0.1524" layer="16"/>
 <wire x1="79.6925" y1="32.0675" x2="80.645" y2="32.0675" width="0.1524" layer="16"/>
+<polygon width="0.1524" layer="16">
+<vertex x="82.55" y="7.3025"/>
+<vertex x="77.1525" y="1.905"/>
+<vertex x="9.525" y="1.905"/>
+<vertex x="3.4925" y="7.9375"/>
+<vertex x="3.4925" y="32.385"/>
+<vertex x="7.9375" y="36.83"/>
+<vertex x="78.4225" y="36.83"/>
+<vertex x="82.55" y="32.7025"/>
+</polygon>
 </signal>
 <signal name="+5V">
@@
 <wire x1="36.5125" y1="29.845" x2="38.735" y2="27.6225" width="0.1524" layer="1"/>
 <wire x1="33.9725" y1="29.845" x2="36.5125" y2="29.845" width="0.1524" layer="1"/>
-<wire x1="13.0175" y1="31.4325" x2="32.385" y2="31.4325" width="0.1524" layer="16"/>
-<wire x1="32.385" y1="31.4325" x2="33.9725" y2="29.845" width="0.1524" layer="16"/>
 <contactref element="IC1" pad="4"/>
 <contactref element="IC2" pad="5"/>
@@
 <wire x1="78.105" y1="22.5425" x2="80.01" y2="24.4475" width="0.1524" layer="1"/>
 <wire x1="80.01" y1="24.4475" x2="80.645" y2="24.4475" width="0.1524" layer="1"/>
+<wire x1="13.0175" y1="31.4325" x2="32.385" y2="31.4325" width="0.1524" layer="1"/>
+<wire x1="32.385" y1="31.4325" x2="33.9725" y2="29.845" width="0.1524" layer="1"/>
 </signal>
 <signal name="SCL">
@@
 <wire x1="43.18" y1="5.08" x2="48.26" y2="10.16" width="0.1524" layer="16"/>
 <wire x1="48.26" y1="10.16" x2="49.53" y2="10.16" width="0.1524" layer="16"/>
-<wire x1="43.18" y1="5.08" x2="37.465" y2="10.795" width="0.1524" layer="16"/>
-<wire x1="37.465" y1="10.795" x2="29.5275" y2="10.795" width="0.1524" layer="16"/>
+<wire x1="43.18" y1="5.08" x2="43.18" y2="6.0325" width="0.1524" layer="16"/>
+<wire x1="43.18" y1="6.0325" x2="38.4175" y2="10.795" width="0.1524" layer="16"/>
+<wire x1="38.4175" y1="10.795" x2="29.5275" y2="10.795" width="0.1524" layer="16"/>
 <wire x1="29.5275" y1="10.795" x2="26.9875" y2="10.795" width="0.1524" layer="16"/>
 <wire x1="26.9875" y1="10.795" x2="24.765" y2="8.5725" width="0.1524" layer="16"/>
@@
 <contactref element="IC1" pad="14"/>
 <contactref element="R2G" pad="2"/>
-<wire x1="70.1675" y1="21.9075" x2="73.025" y2="21.9075" width="0" layer="19" extent="1-1"/>
+<wire x1="73.025" y1="21.9075" x2="70.1675" y2="21.9075" width="0.1524" layer="16"/>
 </signal>
 <signal name="GP13">
 <contactref element="IC1" pad="13"/>
 <contactref element="R2F" pad="2"/>
-<wire x1="70.1675" y1="24.4475" x2="73.025" y2="24.4475" width="0" layer="19" extent="1-1"/>
+<wire x1="73.025" y1="24.4475" x2="70.1675" y2="24.4475" width="0.1524" layer="16"/>
 </signal>
 <signal name="GP12">
 <contactref element="IC1" pad="12"/>
 <contactref element="R3AB" pad="2"/>
-<wire x1="70.1675" y1="26.9875" x2="73.025" y2="26.9875" width="0" layer="19" extent="1-1"/>
+<contactref element="R3AB1" pad="2"/>
+<wire x1="70.1675" y1="29.5275" x2="70.1675" y2="26.9875" width="0.1524" layer="16"/>
+<wire x1="73.025" y1="26.9875" x2="70.1675" y2="26.9875" width="0.1524" layer="16"/>
 </signal>
 <signal name="GP11">
 <contactref element="IC1" pad="11"/>
 <contactref element="R2A" pad="2"/>
-<wire x1="73.025" y1="29.5275" x2="70.1675" y2="29.5275" width="0.1524" layer="16"/>
+<wire x1="73.025" y1="29.5275" x2="70.485" y2="32.0675" width="0.1524" layer="16"/>
+<wire x1="70.485" y1="32.0675" x2="70.1675" y2="32.0675" width="0.1524" layer="16"/>
 </signal>
 <signal name="GP10">
 <contactref element="IC1" pad="10"/>
 <contactref element="R2B" pad="2"/>
-<wire x1="73.025" y1="32.0675" x2="70.1675" y2="32.0675" width="0.1524" layer="16"/>
+<wire x1="73.025" y1="32.0675" x2="70.485" y2="34.6075" width="0.1524" layer="16"/>
+<wire x1="70.485" y1="34.6075" x2="70.1675" y2="34.6075" width="0.1524" layer="16"/>
 </signal>
 <signal name="GP27">
 <contactref element="IC2" pad="17"/>
 <contactref element="R2DP" pad="1"/>
-<wire x1="13.0175" y1="28.8925" x2="15.24" y2="28.8925" width="0" layer="19" extent="1-1"/>
+<wire x1="13.0175" y1="28.8925" x2="15.24" y2="28.8925" width="0.1524" layer="1"/>
 </signal>
 <signal name="GP26">
@@
 <contactref element="R2A" pad="1"/>
 <contactref element="LED2" pad="21"/>
-<wire x1="62.5475" y1="29.5275" x2="60.6425" y2="31.4325" width="0.1524" layer="16"/>
-<wire x1="60.6425" y1="31.4325" x2="43.18" y2="31.4325" width="0.1524" layer="16"/>
-<wire x1="43.18" y1="31.4325" x2="41.5925" y2="29.845" width="0.1524" layer="16"/>
+<wire x1="62.5475" y1="32.0675" x2="61.595" y2="33.02" width="0.1524" layer="16"/>
+<wire x1="61.595" y1="33.02" x2="44.7675" y2="33.02" width="0.1524" layer="16"/>
+<wire x1="44.7675" y1="33.02" x2="41.5925" y2="29.845" width="0.1524" layer="16"/>
 </signal>
 <signal name="N$9">
 <contactref element="R2B" pad="1"/>
 <contactref element="LED2" pad="20"/>
-<wire x1="62.5475" y1="32.0675" x2="61.9125" y2="32.7025" width="0.1524" layer="16"/>
-<wire x1="61.9125" y1="32.7025" x2="41.91" y2="32.7025" width="0.1524" layer="16"/>
-<wire x1="41.91" y1="32.7025" x2="39.0525" y2="29.845" width="0.1524" layer="16"/>
+<wire x1="62.5475" y1="34.6075" x2="43.815" y2="34.6075" width="0.1524" layer="16"/>
+<wire x1="43.815" y1="34.6075" x2="39.0525" y2="29.845" width="0.1524" layer="16"/>
 </signal>
 <signal name="N$10">
@@
 <contactref element="R3AB" pad="1"/>
 <contactref element="LED2" pad="25"/>
-<contactref element="LED2" pad="24"/>
-<wire x1="49.2125" y1="29.845" x2="51.7525" y2="29.845" width="0.1524" layer="16"/>
 <wire x1="51.7525" y1="29.845" x2="54.61" y2="26.9875" width="0.1524" layer="16"/>
 <wire x1="54.61" y1="26.9875" x2="62.5475" y2="26.9875" width="0.1524" layer="16"/>
 </signal>
+<signal name="N$16">
+<contactref element="LED2" pad="24"/>
+<contactref element="R3AB1" pad="1"/>
+<wire x1="62.5475" y1="29.5275" x2="60.6425" y2="31.4325" width="0.1524" layer="16"/>
+<wire x1="60.6425" y1="31.4325" x2="50.8" y2="31.4325" width="0.1524" layer="16"/>
+<wire x1="50.8" y1="31.4325" x2="49.2125" y2="29.845" width="0.1524" layer="16"/>
+</signal>
 </signals>

Commit message: fin des carte tdb
Parts:
- moved C2 3.84 mm to (54.3, 8.57)
- moved C3 1.80 mm to (54.6, 3.81), turned to 180 degrees
- moved C1 1.59 mm to (33.7, 3.17), turned to 0 degrees
- renumbered R3AB to R3A, R3AB1 to R3B
Routing:
- net GND: track 130.7 -> 0.00 mm
- net SCL: track 101.7 -> 103.6 mm
- net SDA: track 101.3 -> 103.0 mm
- net +5V: track 143.4 -> 142.5 mm
