File: EL - Electrical/Autre/BSPD/Version FSG/FSG_2019_BSPD_0.2_traversant.sch (EAGLE design)
At the start: 48 parts, among them IC1 LM393N, IC2 LM393N, IC3 LM393N, K101 CP1-12V, T101 Si2309CDS, T102 BSS138, T103 BSS138

Commit message: BSPD traversant
Parts:
- removed C101, C105: 100n, resistor:C-EUC0603
- removed C103, C106, C108: 10µ, rcl:C-EUC1206
- removed C104: 10µ, rcl:C-EUC1206K
- removed C107, C109, C110: 100n, rcl:C-EUC0603
- removed I104: SN74AUC1G02DBVR, Arduino:NC7SZ08M5X
- removed I105: LM1117MPX-5.0, IntegratedCircuits:0022_LM1117IMPX-5.0
- added C1, C4, C6, C7: 10u, rcl:C-EU075-052X106
- added C2, C3, C5, C8, C9: 100n, rcl:C-EU025-024X044
- added IC4: SN75452BP, texas-sn55-sn75:SN75452BP
- added IC5: (no value), v-reg-3:LM1117V
Connections:
- net +12V: now also C2.1, C4.1, IC5.IN; no longer C106.1, C107.1, I105.IN
- net +5V: now also C1.1, C3.1, C5.1, C6.1, C8.1, C9.1, IC4P.VCC, IC5.OUT; no longer C101.2, C104.1, C105.2, C108.1, C109.2, C110.1, I104.VCC, I105.OUT, I105.OUT@1
- net GND: now also C1.2, C2.2, C3.2, C4.2, C7.2, C8.2, C9.2, IC4P.GND, IC5.GND; no longer C101.1, C103.2, C105.1, C106.2, C107.2, C108.2, C109.1, I104.GND, I105.GND/ADJ
- net N$17: now also C7.1; no longer C103.1
- net N$2: now also IC4A.I1; no longer I104.B
- net N$3: now also IC4A.O; no longer I104.Y
- net N$5: now also C5.2; no longer C110.2
- net N$7: now also C6.2; no longer C104.2
- net N$9: now also IC4A.I0; no longer I104.A
