File: EL - Electrical/Autre/BSPD/Version FSG/FSG_2019_BSPD_0.2_SMD.brd (EAGLE design)
At the start: 44 x 36 mm, 49 parts, among them K101 CP1-12V, T101 Si2309CDS, T102 BSS138, T103 BSS138

Commit message: Mofif connecteur BSPD
Parts:
- removed JP1: (no value), pinhead:1X06
- added J1: 22-05-7068-06, con-molex:7395-06
Connections:
- net +12V: now also J1.6; no longer JP1.1
- net GND: now also J1.1; no longer JP1.6
- net SC_IN: now also J1.5; no longer JP1.2
- net SC_OUT: now also J1.4; no longer JP1.3
- net SENS_1: now also J1.3; no longer JP1.4
- net SENS_2: now also J1.2; no longer JP1.5
Routing:
- net +12V: track 47.4 -> 44.9 mm
- net SENS_1: track 19.6 -> 18.5 mm
- net SENS_2: track 12.6 -> 11.4 mm
- net SC_OUT: track 12.0 -> 10.9 mm
- net SC_IN: track 12.4 -> 11.3 mm
