File: EL - Electrical/Autre/Carte avant/Shield carte avant/shield carte avant.sch (EAGLE design)
At the start: 14 parts, among them J5 22-05-7028-02

Commit message: shield carte avant
Parts:
- added J1: 22-05-7108-10, con-molex:22-05-7108-10
Connections:
- new net N$11: J1-7.S
- new net N$12: J1-8.S
- new net N$13: J1-9.S
- new net N$14: J1-10.S
- new net N$6: J1-2.S
- new net N$7: J1-3.S
- new net N$8: J1-4.S
- new net N$9: J1-5.S
- net 12V: now also C4.2
- net 5V: now also J1-1.S, J1-6.S
Other:
- note removed: "EPSA - Ecurie Piston Sport Auto Vulcanix 2017/2018"
- moved on the sheet: ANALOGIN, C3, C4, DIGITALIN0_7, DIGITALIN8_13, POWER, PS1

Commit message: maj shield carte avant
Parts:
- removed PS1: THN_15-1211, THN_15-1211:THN_15-1211
- added D2: 1N5819-B, diode:1N5819-B
- added IC1: LM2576T, v-reg-3:LM2576T
- added L1: 100uH, wurth_elektronik_passive_rev16d:WE-TI_8012
- C4: value 470pF -> 100uF
Connections:
- removed net N$14: J1-10.S
- net 12V: no longer C4.2
- net 5V: now also C3.2, IC1.FB, J1-10.S, L1.2; no longer C4.1, PS1.+_VOUT
- net GND: now also C4.1, D2.A, IC1.GND, IC1.OFF, J5-2.S; no longer J5-1.S, PS1.-VIN_(GND), PS1.REMOTE_ON/OFF
- net N$1: now also J5-1.S; no longer J5-2.S
- net N$2: now also D2.C, IC1.OUT, L1.1; no longer C3.2, PS1.-VOUT
- net N$3: now also C4.2, IC1.VIN; no longer PS1.+VIN_(VCC)
Other:
- note added: "Connection extérieur"
- moved on the sheet: C3, C4, J5-1, J5-2

Commit message: légère modifs à terminer
Connections:
- removed net N$11: J1-7.S
- removed net N$12: J1-8.S
- removed net N$13: J1-9.S
- removed net N$6: J1-2.S
- removed net N$7: J1-3.S
- removed net N$8: J1-4.S
- removed net N$9: J1-5.S
- new net A4: ANALOGIN.4, J1-9.S
- new net A5: ANALOGIN.5, J1-10.S
- new net D1: DIGITALIN0_7.1, J1-1.S
- new net D2: DIGITALIN0_7.2, J1-2.S
- new net D3: DIGITALIN0_7.3, J1-3.S
- new net D4: DIGITALIN0_7.4, J1-4.S
- new net D5: DIGITALIN0_7.5, J1-5.S
- new net D6: DIGITALIN0_7.6, J1-6.S
- new net D7: DIGITALIN0_7.7, J1-7.S
- net 5V: now also J1-8.S; no longer J1-1.S, J1-10.S, J1-6.S
Changed lines of the file:
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@@
 <wire x1="-144.78" y1="157.48" x2="-144.78" y2="228.6" width="0.1524" layer="249"/>
 <text x="-142.24" y="223.52" size="2.54" layer="249">ALIMENTATION 12V</text>
-<wire x1="-157.48" y1="68.58" x2="-91.44" y2="68.58" width="0.1524" layer="249"/>
-<wire x1="-91.44" y1="68.58" x2="-91.44" y2="-5.08" width="0.1524" layer="249"/>
-<wire x1="-91.44" y1="-5.08" x2="-157.48" y2="-5.08" width="0.1524" layer="249"/>
+<wire x1="-157.48" y1="68.58" x2="-86.36" y2="68.58" width="0.1524" layer="249"/>
+<wire x1="-86.36" y1="68.58" x2="-86.36" y2="-5.08" width="0.1524" layer="249"/>
+<wire x1="-86.36" y1="-5.08" x2="-157.48" y2="-5.08" width="0.1524" layer="249"/>
 <wire x1="-157.48" y1="-5.08" x2="-157.48" y2="68.58" width="0.1524" layer="249"/>
 <text x="-144.78" y="63.5" size="2.54" layer="249">Connection Pins Arduino</text>
@@
 <net name="5V" class="0">
 <segment>
-<pinref part="J1" gate="-1" pin="S"/>
-<wire x1="-38.1" y1="50.8" x2="-45.72" y2="50.8" width="0.1524" layer="91"/>
-</segment>
-<segment>
-<pinref part="J1" gate="-6" pin="S"/>
-<wire x1="-38.1" y1="25.4" x2="-45.72" y2="25.4" width="0.1524" layer="91"/>
-</segment>
-<segment>
 <pinref part="IC1" gate="A" pin="FB"/>
 <wire x1="-81.28" y1="121.92" x2="-45.72" y2="121.92" width="0.1524" layer="91"/>
@@
 </segment>
 <segment>
-<pinref part="J1" gate="-10" pin="S"/>
-<wire x1="-38.1" y1="5.08" x2="-45.72" y2="5.08" width="0.1524" layer="91"/>
-<label x="-45.72" y="5.08" size="1.778" layer="95" rot="R180" xref="yes"/>
-</segment>
-</net>
-<net name="N$6" class="0">
-<segment>
-<pinref part="J1" gate="-2" pin="S"/>
-<wire x1="-38.1" y1="45.72" x2="-45.72" y2="45.72" width="0.1524" layer="91"/>
-</segment>
-</net>
-<net name="N$7" class="0">
+<pinref part="J1" gate="-8" pin="S"/>
+<wire x1="-38.1" y1="15.24" x2="-45.72" y2="15.24" width="0.1524" layer="91"/>
+<label x="-45.72" y="15.24" size="1.778" layer="95" rot="R180" xref="yes"/>
+</segment>
+</net>
+<net name="D6" class="0">
+<segment>
+<pinref part="DIGITALIN0_7" gate="A" pin="6"/>
+<label x="-93.98" y="25.4" size="1.778" layer="95" xref="yes"/>
+<wire x1="-111.76" y1="25.4" x2="-93.98" y2="25.4" width="0.1524" layer="91"/>
+</segment>
+<segment>
+<pinref part="J1" gate="-6" pin="S"/>
+<wire x1="-38.1" y1="25.4" x2="-45.72" y2="25.4" width="0.1524" layer="91"/>
+<label x="-45.72" y="25.4" size="1.778" layer="95" rot="R180" xref="yes"/>
+</segment>
+</net>
+<net name="D5" class="0">
+<segment>
+<pinref part="DIGITALIN0_7" gate="A" pin="5"/>
+<wire x1="-111.76" y1="22.86" x2="-104.14" y2="22.86" width="0.1524" layer="91"/>
+<label x="-104.14" y="22.86" size="1.778" layer="95" xref="yes"/>
+</segment>
+<segment>
+<pinref part="J1" gate="-5" pin="S"/>
+<wire x1="-38.1" y1="30.48" x2="-45.72" y2="30.48" width="0.1524" layer="91"/>
+<label x="-45.72" y="30.48" size="1.778" layer="95" rot="R180" xref="yes"/>
+</segment>
+</net>
+<net name="D4" class="0">
+<segment>
+<pinref part="J1" gate="-4" pin="S"/>
+<wire x1="-38.1" y1="35.56" x2="-45.72" y2="35.56" width="0.1524" layer="91"/>
+<label x="-45.72" y="35.56" size="1.778" layer="95" rot="R180" xref="yes"/>
+</segment>
+<segment>
+<pinref part="DIGITALIN0_7" gate="A" pin="4"/>
+<label x="-93.98" y="20.32" size="1.778" layer="95" xref="yes"/>
+<wire x1="-93.98" y1="20.32" x2="-111.76" y2="20.32" width="0.1524" layer="91"/>
+</segment>
+</net>
+<net name="D3" class="0">
+<segment>
+<pinref part="DIGITALIN0_7" gate="A" pin="3"/>
+<wire x1="-111.76" y1="17.78" x2="-104.14" y2="17.78" width="0.1524" layer="91"/>
+<label x="-104.14" y="17.78" size="1.778" layer="95" xref="yes"/>
+</segment>
 <segment>
 <pinref part="J1" gate="-3" pin="S"/>
 <wire x1="-38.1" y1="40.64" x2="-45.72" y2="40.64" width="0.1524" layer="91"/>
-</segment>
-</net>
-<net name="N$8" class="0">
-<segment>
-<pinref part="J1" gate="-4" pin="S"/>
-<wire x1="-38.1" y1="35.56" x2="-45.72" y2="35.56" width="0.1524" layer="91"/>
-</segment>
-</net>
-<net name="N$9" class="0">
-<segment>
-<pinref part="J1" gate="-5" pin="S"/>
-<wire x1="-38.1" y1="30.48" x2="-45.72" y2="30.48" width="0.1524" layer="91"/>
-</segment>
-</net>
-<net name="N$11" class="0">
-<segment>
-<pinref part="J1" gate="-7" pin="S"/>
-<wire x1="-38.1" y1="20.32" x2="-45.72" y2="20.32" width="0.1524" layer="91"/>
-</segment>
-</net>
-<net name="N$12" class="0">
-<segment>
-<pinref part="J1" gate="-8" pin="S"/>
-<wire x1="-38.1" y1="15.24" x2="-45.72" y2="15.24" width="0.1524" layer="91"/>
-</segment>
-</net>
-<net name="N$13" class="0">
+<label x="-45.72" y="40.64" size="1.778" layer="95" rot="R180" xref="yes"/>
+</segment>
+</net>
+<net name="D1" class="0">
+<segment>
+<pinref part="DIGITALIN0_7" gate="A" pin="1"/>
+<wire x1="-111.76" y1="12.7" x2="-104.14" y2="12.7" width="0.1524" layer="91"/>
+<label x="-104.14" y="12.7" size="1.778" layer="95" xref="yes"/>
+</segment>
+<segment>
+<pinref part="J1" gate="-1" pin="S"/>
+<wire x1="-38.1" y1="50.8" x2="-45.72" y2="50.8" width="0.1524" layer="91"/>
+<label x="-45.72" y="50.8" size="1.778" layer="95" rot="R180" xref="yes"/>
+</segment>
+</net>
+<net name="A4" class="0">
 <segment>
 <pinref part="J1" gate="-9" pin="S"/>
 <wire x1="-38.1" y1="10.16" x2="-45.72" y2="10.16" width="0.1524" layer="91"/>
+<label x="-45.72" y="10.16" size="1.778" layer="95" rot="R180" xref="yes"/>
+</segment>
+<segment>
+<pinref part="ANALOGIN" gate="A" pin="4"/>
+<wire x1="-134.62" y1="22.86" x2="-142.24" y2="22.86" width="0.1524" layer="91"/>
+<label x="-142.24" y="22.86" size="1.778" layer="95" rot="R180" xref="yes"/>
 </segment>
 </net>
@@
 </segment>
 </net>
+<net name="A5" class="0">
+<segment>
+<pinref part="J1" gate="-10" pin="S"/>
+<wire x1="-38.1" y1="5.08" x2="-45.72" y2="5.08" width="0.1524" layer="91"/>
+<label x="-45.72" y="5.08" size="1.778" layer="95" rot="R180" xref="yes"/>
+</segment>
+<segment>
+<pinref part="ANALOGIN" gate="A" pin="5"/>
+<label x="-149.86" y="25.4" size="1.778" layer="95" rot="R180" xref="yes"/>
+<wire x1="-134.62" y1="25.4" x2="-149.86" y2="25.4" width="0.1524" layer="91"/>
+</segment>
+</net>
+<net name="D2" class="0">
+<segment>
+<pinref part="DIGITALIN0_7" gate="A" pin="2"/>
+<label x="-93.98" y="15.24" size="1.778" layer="95" xref="yes"/>
+<wire x1="-93.98" y1="15.24" x2="-111.76" y2="15.24" width="0.1524" layer="91"/>
+</segment>
+<segment>
+<pinref part="J1" gate="-2" pin="S"/>
+<wire x1="-38.1" y1="45.72" x2="-45.72" y2="45.72" width="0.1524" layer="91"/>
+<label x="-45.72" y="45.72" size="1.778" layer="95" rot="R180" xref="yes"/>
+</segment>
+</net>
+<net name="D7" class="0">
+<segment>
+<pinref part="DIGITALIN0_7" gate="A" pin="7"/>
+<wire x1="-111.76" y1="27.94" x2="-104.14" y2="27.94" width="0.1524" layer="91"/>
+<label x="-104.14" y="27.94" size="1.778" layer="95" xref="yes"/>
+</segment>
+<segment>
+<pinref part="J1" gate="-7" pin="S"/>
+<wire x1="-38.1" y1="20.32" x2="-45.72" y2="20.32" width="0.1524" layer="91"/>
+<label x="-45.72" y="20.32" size="1.778" layer="95" rot="R180" xref="yes"/>
+</segment>
+</net>

Commit message: mAj du shield avant
Parts:
- removed ANALOGIN, POWER: (no value), carduino:PINHD-1X6CB
- removed D2: 1N5819-B, diode:1N5819-B
- removed DIGITALIN0_7, DIGITALIN8_13: (no value), carduino:PINHD-1X8CLEANBIG
- removed L1: 100uH, wurth_elektronik_passive_rev16d:WE-TI_8012
- added C5: 680 pF, rcl:C-EU025-024X044
- added IC2: MCP2515-I_SO, MCP2515-I_SO:MCP2515-I_SO
- added J2: 22-05-7028-02, con-molex:22-05-7028-02
- added J3: 22-05-7038-03, con-molex:22-05-7038-03
- added M1: ARDUINO_R3_ICSP, adafruit:ARDUINO_R3_ICSP
- added PS1: THN_15-1211, THN_15-1211:THN_15-1211
- added QUARTZ_16_MHZ: FOXSLF_160-20, FOXSLF_160-20:FOXSLF_160-20
- added R1, R3: 1k, rcl:R-EU_0204/7
- added R2: 120, rcl:R-EU_0204/7
- added SW1: (no value), adafruit:SWITCH_PUSHBUTTONEVQ-PE
- C3: value 470pF -> 4.7 uF; device rcl:C-EU025-025X050 -> rcl:C-EU025-024X044
- C4: value 100uF -> 680 pF; device rcl:C-EU025-025X050 -> rcl:C-EU025-024X044
- IC1: value LM2576T -> MCP2562-E_SN; device v-reg-3:LM2576T -> MCP2562-E_SN:MCP2562-E_SN
- J1: value 22-05-7108-10 -> 22-05-7078-07; device con-molex:22-05-7108-10 -> con-molex:22-05-7078-07
Connections:
- removed net 5V: C3.2, IC1.FB, J1-8.S, L1.2
- removed net N$2: D2.C, IC1.OUT, L1.1
- new net +5_V: C4.1, IC1.VDD, IC2.VDD, J1-5.S, PS1.+_VOUT
- new net CS: IC2.!CS, M1.D10
- new net INT: IC2.!INT, M1.D2
- new net N$10: IC2.OSC2, QUARTZ_16_MHZ.2
- new net N$11: IC2.OSC1, QUARTZ_16_MHZ.1
- new net N$13: M1.GND@2
- new net N$14: R3.1, SW1.P$2
- new net N$15: IC2.!RESET, R3.2
- new net N$16: M1.GND@1
- new net N$5: IC1.TXD, IC2.TXCAN
- new net N$6: IC1.RXD, IC2.RXCAN
- new net N$7: IC1.VSS, R1.2
- new net N$8: IC1.CANH, J2-1.S, R2.2
- new net N$9: IC1.CANL, J2-2.S, R2.1
- new net RESET: M1./RESET, SW1.P$1
- new net RIEN: M1.5V
- new net SCK: IC2.SCK, M1.SCK
- new net SI: IC2.SI, M1.MOSI
- new net SO: IC2.SO, M1.MISO
- net 12V: now also C3.1, C4.2, PS1.+VIN_(VCC)
- net A4: now also J1-6.S; no longer ANALOGIN.4, J1-9.S
- net A5: now also J1-7.S; no longer ANALOGIN.5, J1-10.S
- net D1: now also J3-1.S; no longer DIGITALIN0_7.1, J1-1.S
- net D2: now also J3-2.S; no longer DIGITALIN0_7.2, J1-2.S
- net D3: now also J3-3.S; no longer DIGITALIN0_7.3, J1-3.S
- net D4: now also J1-1.S; no longer DIGITALIN0_7.4, J1-4.S
- net D5: now also J1-2.S; no longer DIGITALIN0_7.5, J1-5.S
- net D6: now also J1-3.S; no longer DIGITALIN0_7.6, J1-6.S
- net D7: now also J1-4.S; no longer DIGITALIN0_7.7, J1-7.S
- net GND: now also C3.2, C5.2, IC2.VSS, PS1.-VIN_(GND), R1.1; no longer C3.1, C4.1, D2.A, IC1.GND, IC1.OFF
- net N$3: now also C5.1, PS1.-VOUT; no longer C4.2, IC1.VIN
Other:
- moved on the sheet: ALIM_ARDUINO-1, ALIM_ARDUINO-2, C1, C2, C3, C4, D1, F1, J1-1, J1-2, J1-3, J1-4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
