File: EL - Electrical/Autre/Carte avant/Shield carte avant/shield carte avant.brd (EAGLE design)
At the start: 69.2 x 53.4 mm, 14 parts, among them J5 22-05-7028-02

Commit message: shield carte avant
Parts:
- added J1: 22-05-7108-10, con-molex:7395-10
- moved C3 14.5 mm to (21.6, 38.1)
- moved F1 13.2 mm to (14.1, 38.4), turned to 90 degrees
- moved PS1 11.7 mm to (24.1, 35.6)
- moved C2 6.71 mm to (21.0, 22.5), turned to 90 degrees
- moved C4 6.35 mm to (52.1, 31.8), turned to 270 degrees
- moved C1 6.35 mm to (10.8, 15.5)
- moved R20 4.02 mm to (27.3, 6.99), turned to 0 degrees
- moved J5 3.81 mm to (6.22, 37.7)
- moved D1 2.54 mm to (22.6, 3.05)
Connections:
- new net N$11: J1.7
- new net N$12: J1.8
- new net N$13: J1.9
- new net N$14: J1.10
- new net N$6: J1.2
- new net N$7: J1.3
- new net N$8: J1.4
- new net N$9: J1.5
- net 12V: now also C4.2
- net 5V: now also J1.1, J1.6
Routing:
- net 12V: track 0.00 -> 101.1 mm
- net GND: track 0.00 -> 89.5 mm
- net 5V: track 0.00 -> 17.1 mm
- net N$1: track 0.00 -> 13.9 mm
- net N$2: track 0.00 -> 9.89 mm
- net N$4: track 0.00 -> 7.60 mm
Other:
- outline, holes or cut-outs redrawn

Commit message: maj shield carte avant
Parts:
- removed PS1: THN_15-1211, THN_15-1211:THN-15-SERIES
- added D2: 1N5819-B, diode:DO41-7.6
- added IC1: LM2576T, v-reg-3:TO220-5
- added L1: 100uH, wurth_elektronik_passive_rev16d:WE-TI_8012
- C4: value 470pF -> 100uF
- moved C4 22.5 mm to (30.5, 25.4), turned to 0 degrees
- moved C3 10.9 mm to (30.5, 31.8), turned to 0 degrees
- turned F1 to 270 degrees
Connections:
- removed net N$14: J1.10
- net 12V: no longer C4.2
- net 5V: now also C3.2, IC1.4, J1.10, L1.2; no longer C4.1, PS1.3
- net GND: now also C4.1, D2.A, IC1.3, IC1.5, J5.2; no longer J5.1, PS1.2, PS1.6
- net N$1: now also J5.1; no longer J5.2
- net N$2: now also D2.C, IC1.2, L1.1; no longer C3.2, PS1.5
- net N$3: now also C4.2, IC1.1; no longer PS1.1
Routing:
- net 12V: track 101.1 -> 42.4 mm
- net 5V: track 17.1 -> 69.9 mm
- net GND: track 89.5 -> 100.5 mm
- net N$3: track 0.00 -> 5.93 mm
- net N$2: track 9.89 -> 14.4 mm
- net N$1: track 13.9 -> 15.1 mm

Commit message: légère modifs à terminer
Connections:
- removed net N$11: J1.7
- removed net N$12: J1.8
- removed net N$13: J1.9
- removed net N$6: J1.2
- removed net N$7: J1.3
- removed net N$8: J1.4
- removed net N$9: J1.5
- new net A4: ANALOGIN.4, J1.9
- new net A5: ANALOGIN.5, J1.10
- new net D1: DIGITALIN0_7.1, J1.1
- new net D2: DIGITALIN0_7.2, J1.2
- new net D3: DIGITALIN0_7.3, J1.3
- new net D4: DIGITALIN0_7.4, J1.4
- new net D5: DIGITALIN0_7.5, J1.5
- new net D6: DIGITALIN0_7.6, J1.6
- new net D7: DIGITALIN0_7.7, J1.7
- net 5V: now also J1.8; no longer J1.1, J1.10, J1.6
Routing:
- net D7: track 0.00 -> 27.8 mm
- net D6: track 0.00 -> 24.2 mm
- net A4: track 0.00 -> 23.5 mm
- net D5: track 0.00 -> 20.6 mm
- net A5: track 0.00 -> 19.9 mm
- net D4: track 0.00 -> 17.0 mm
- net D3: track 0.00 -> 13.4 mm
- net D2: track 0.00 -> 9.84 mm
- net D1: track 0.00 -> 6.51 mm
- net 5V: track 69.9 -> 72.0 mm
- added copper zone on layer 1, net GND
Changed lines of the file:
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@@
 <wire x1="20.955" y1="28.575" x2="20.955" y2="23.749" width="1.016" layer="1"/>
 <wire x1="13.081" y1="36.449" x2="20.955" y2="28.575" width="1.016" layer="1"/>
+<polygon width="1.016" layer="1">
+<vertex x="3.81" y="52.07"/>
+<vertex x="64.77" y="52.07"/>
+<vertex x="67.31" y="49.53"/>
+<vertex x="66.04" y="48.26"/>
+<vertex x="66.04" y="3.81"/>
+<vertex x="63.5" y="1.27"/>
+<vertex x="5.08" y="1.27"/>
+<vertex x="2.54" y="3.81"/>
+<vertex x="2.54" y="50.8"/>
+</polygon>
 </signal>
 <signal name="12V" class="1">
@@
 </signal>
 <signal name="5V">
-<contactref element="J1" pad="1"/>
-<contactref element="J1" pad="6"/>
 <contactref element="IC1" pad="4"/>
 <contactref element="C3" pad="2"/>
@@
 <wire x1="27.51" y1="15.93" x2="34.51" y2="8.93" width="0.6096" layer="1"/>
 <wire x1="34.51" y1="8.93" x2="40.64" y2="8.93" width="0.6096" layer="1"/>
-<contactref element="J1" pad="10"/>
-<wire x1="53.3" y1="21.59" x2="63.5" y2="21.59" width="1.016" layer="1"/>
 <wire x1="40.64" y1="8.93" x2="53.3" y2="21.59" width="1.016" layer="1"/>
 <wire x1="31.75" y1="31.75" x2="43.18" y2="31.75" width="0.6096" layer="1"/>
 <wire x1="43.18" y1="31.75" x2="53.3" y2="21.63" width="0.6096" layer="1"/>
 <wire x1="53.3" y1="21.63" x2="53.3" y2="21.59" width="0.6096" layer="1"/>
-<wire x1="63.5" y1="31.75" x2="63.5" y2="44.45" width="0" layer="19" extent="1-1"/>
-<wire x1="63.5" y1="21.59" x2="63.5" y2="31.75" width="0" layer="19" extent="1-1"/>
+<contactref element="J1" pad="8"/>
+<wire x1="53.3" y1="21.63" x2="58.34" y2="26.67" width="1.016" layer="1"/>
+<wire x1="58.34" y1="26.67" x2="63.5" y2="26.67" width="1.016" layer="1"/>
 </signal>
-<signal name="N$6">
-<contactref element="J1" pad="2"/>
+<signal name="D6">
+<contactref element="DIGITALIN0_7" pad="6"/>
+<contactref element="J1" pad="6"/>
+<wire x1="63.5" y1="31.75" x2="62.2808" y2="32.9692" width="0.6096" layer="1"/>
+<wire x1="62.2808" y1="32.9692" x2="62.19090625" y2="32.9692" width="0.6096" layer="1"/>
+<wire x1="62.19090625" y1="32.9692" x2="51.181" y2="43.97910625" width="0.6096" layer="1"/>
+<wire x1="51.181" y1="43.97910625" x2="51.181" y2="50.8" width="0.6096" layer="1"/>
 </signal>
-<signal name="N$7">
+<signal name="D5">
+<contactref element="DIGITALIN0_7" pad="5"/>
+<contactref element="J1" pad="5"/>
+<wire x1="62.19090625" y1="35.5092" x2="62.2808" y2="35.5092" width="0.6096" layer="1"/>
+<wire x1="62.2808" y1="35.5092" x2="63.5" y2="34.29" width="0.6096" layer="1"/>
+<wire x1="53.721" y1="50.8" x2="53.721" y2="43.97910625" width="0.6096" layer="1"/>
+<wire x1="53.721" y1="43.97910625" x2="62.19090625" y2="35.5092" width="0.6096" layer="1"/>
+</signal>
+<signal name="D4">
+<contactref element="J1" pad="4"/>
+<contactref element="DIGITALIN0_7" pad="4"/>
+<wire x1="63.5" y1="36.83" x2="62.2808" y2="38.0492" width="0.6096" layer="1"/>
+<wire x1="62.2808" y1="38.0492" x2="62.19090625" y2="38.0492" width="0.6096" layer="1"/>
+<wire x1="62.19090625" y1="38.0492" x2="56.261" y2="43.97910625" width="0.6096" layer="1"/>
+<wire x1="56.261" y1="43.97910625" x2="56.261" y2="50.8" width="0.6096" layer="1"/>
+</signal>
+<signal name="D3">
+<contactref element="DIGITALIN0_7" pad="3"/>
 <contactref element="J1" pad="3"/>
+<wire x1="62.19090625" y1="40.5892" x2="62.2808" y2="40.5892" width="0.6096" layer="1"/>
+<wire x1="62.2808" y1="40.5892" x2="63.5" y2="39.37" width="0.6096" layer="1"/>
+<wire x1="58.801" y1="50.8" x2="58.801" y2="43.97910625" width="0.6096" layer="1"/>
+<wire x1="58.801" y1="43.97910625" x2="62.19090625" y2="40.5892" width="0.6096" layer="1"/>
 </signal>
-<signal name="N$8">
-<contactref element="J1" pad="4"/>
+<signal name="D1">
+<contactref element="DIGITALIN0_7" pad="1"/>
+<contactref element="J1" pad="1"/>
+<wire x1="63.5" y1="44.45" x2="63.5" y2="50.419" width="0.6096" layer="1"/>
+<wire x1="63.5" y1="50.419" x2="63.881" y2="50.8" width="0.6096" layer="1"/>
 </signal>
-<signal name="N$9">
-<contactref element="J1" pad="5"/>
-</signal>
-<signal name="N$11">
-<contactref element="J1" pad="7"/>
-</signal>
-<signal name="N$12">
-<contactref element="J1" pad="8"/>
-</signal>
-<signal name="N$13">
+<signal name="A4">
 <contactref element="J1" pad="9"/>
+<contactref element="ANALOGIN" pad="4"/>
+<wire x1="62.19090625" y1="22.9108" x2="62.2808" y2="22.9108" width="0.6096" layer="1"/>
+<wire x1="62.2808" y1="22.9108" x2="63.5" y2="24.13" width="0.6096" layer="1"/>
+<wire x1="58.928" y1="2.54" x2="58.928" y2="19.64789375" width="0.6096" layer="1"/>
+<wire x1="58.928" y1="19.64789375" x2="62.19090625" y2="22.9108" width="0.6096" layer="1"/>
 </signal>
 <signal name="N$3">
@@
 <wire x1="14.097" y1="46.863" x2="14.097" y2="50.8762" width="1.016" layer="1"/>
 </signal>
+<signal name="A5">
+<contactref element="J1" pad="10"/>
+<contactref element="ANALOGIN" pad="5"/>
+<wire x1="61.468" y1="2.54" x2="61.468" y2="19.558" width="0.6096" layer="1"/>
+<wire x1="61.468" y1="19.558" x2="63.5" y2="21.59" width="0.6096" layer="1"/>
+</signal>
+<signal name="D2">
+<contactref element="DIGITALIN0_7" pad="2"/>
+<contactref element="J1" pad="2"/>
+<wire x1="63.5" y1="41.91" x2="62.2808" y2="43.1292" width="0.6096" layer="1"/>
+<wire x1="62.2808" y1="43.1292" x2="62.19090625" y2="43.1292" width="0.6096" layer="1"/>
+<wire x1="62.19090625" y1="43.1292" x2="61.341" y2="43.97910625" width="0.6096" layer="1"/>
+<wire x1="61.341" y1="43.97910625" x2="61.341" y2="50.8" width="0.6096" layer="1"/>
+</signal>
+<signal name="D7">
+<contactref element="DIGITALIN0_7" pad="7"/>
+<contactref element="J1" pad="7"/>
+<wire x1="62.19090625" y1="30.4292" x2="62.2808" y2="30.4292" width="0.6096" layer="1"/>
+<wire x1="62.2808" y1="30.4292" x2="63.5" y2="29.21" width="0.6096" layer="1"/>
+<wire x1="48.641" y1="50.8" x2="48.641" y2="43.97910625" width="0.6096" layer="1"/>
+<wire x1="48.641" y1="43.97910625" x2="62.19090625" y2="30.4292" width="0.6096" layer="1"/>
+</signal>
 </signals>

Commit message: mAj du shield avant
Parts:
- removed ANALOGIN, POWER: (no value), carduino:1X06-CLEANBIG
- removed D2: 1N5819-B, diode:DO41-7.6
- removed DIGITALIN0_7, DIGITALIN8_13: (no value), carduino:1X08-CLEANBIG
- removed L1: 100uH, wurth_elektronik_passive_rev16d:WE-TI_8012
- added C5: 680 pF, rcl:C025-024X044
- added IC2: MCP2515-I_SO, MCP2515-I_SO:SOIC127P1030X265-18N
- added J2: 22-05-7028-02, con-molex:7395-02
- added J3: 22-05-7038-03, con-molex:7395-03
- added M1: ARDUINO_R3_ICSP, adafruit:ARDUINOR3_ICSP
- added PS1: THN_15-1211, THN_15-1211:THN-15-SERIES
- added QUARTZ_16_MHZ: FOXSLF_160-20, FOXSLF_160-20:HC49SLF_1
- added R1, R3: 1k, rcl:0204/7
- added R2: 120, rcl:0204/7
- added SW1: (no value), adafruit:TACT_PANA-EVQ
- C3: value 470pF -> 4.7 uF; device rcl:C025-025X050 -> rcl:C025-024X044
- C4: value 100uF -> 680 pF; device rcl:C025-025X050 -> rcl:C025-024X044
- IC1: value LM2576T -> MCP2562-E_SN; device v-reg-3:TO220-5 -> MCP2562-E_SN:SOIC127P600X175-8N
- J1: value 22-05-7108-10 -> 22-05-7078-07; device con-molex:7395-10 -> con-molex:7395-07
- moved IC1 31.6 mm to (34.9, 42.5)
- moved C3 17.8 mm to (29.2, 14.0), turned to 180 degrees
- moved J1 17.8 mm to (64.8, 15.2)
- moved R20 4.45 mm to (22.9, 6.99)
- moved C2 3.24 mm to (21.6, 19.3)
- moved C4 1.80 mm to (29.2, 24.1), turned to 180 degrees
- moved D1 1.31 mm to (21.3, 3.37)
Connections:
- removed net 5V: C3.2, IC1.4, J1.8, L1.2
- removed net N$2: D2.C, IC1.2, L1.1
- new net +5_V: C4.1, IC1.3, IC2.18, J1.5, PS1.3
- new net 3V: M1.3V
- new net CS: IC2.16, M1.D10
- new net INT: IC2.12, M1.D2
- new net N$10: IC2.7, QUARTZ_16_MHZ.2
- new net N$11: IC2.8, QUARTZ_16_MHZ.1
- new net N$13: M1.GND@1
- new net N$14: R3.1, SW1.P$2
- new net N$15: IC2.17, R3.2
- new net N$16: M1.GND@3
- new net N$5: IC1.1, IC2.1
- new net N$6: IC1.4, IC2.2
- new net N$7: IC1.2, R1.2
- new net N$8: IC1.7, J2.1, R2.2
- new net N$9: IC1.6, J2.2, R2.1
- new net RESET: M1.RESET, SW1.P$1
- new net RIEN: M1.5V
- new net SCK: IC2.13, M1.SCK
- new net SI: IC2.14, M1.MOSI
- new net SO: IC2.15, M1.MISO
- new net VIN: M1.VIN
- net 12V: now also C3.1, C4.2, PS1.1
- net A4: now also J1.6; no longer ANALOGIN.4, J1.9
- net A5: now also J1.7; no longer ANALOGIN.5, J1.10
- net D1: now also J3.1; no longer DIGITALIN0_7.1, J1.1
- net D2: now also J3.2; no longer DIGITALIN0_7.2, J1.2
- net D3: now also J3.3; no longer DIGITALIN0_7.3, J1.3
- net D4: now also J1.1; no longer DIGITALIN0_7.4, J1.4
- net D5: now also J1.2; no longer DIGITALIN0_7.5, J1.5
- net D6: now also J1.3; no longer DIGITALIN0_7.6, J1.6
- net D7: now also J1.4; no longer DIGITALIN0_7.7, J1.7
- net GND: now also C3.2, C5.2, IC2.9, M1.GND, PS1.2, R1.1; no longer C3.1, C4.1, D2.A, IC1.3, IC1.5
- net N$3: now also C5.1, PS1.5; no longer C4.2, IC1.1
Routing:
- net GND: track 100.5 -> 1.04 mm
- net RESET: track 0.00 -> 98.1 mm
- net +5_V: track 0.00 -> 81.0 mm
- net 5V: track 72.0 -> 0.00 mm
- net 12V: track 42.4 -> 83.4 mm
- net N$8: track 0.00 -> 29.0 mm
- net N$9: track 0.00 -> 28.5 mm
- net D7: track 27.8 -> 0.00 mm
- net SI: track 0.00 -> 27.3 mm
- net D6: track 24.2 -> 0.00 mm
- net A4: track 23.5 -> 0.00 mm
- net SCK: track 0.00 -> 22.2 mm, vias 0 -> 1
- net SO: track 0.00 -> 22.1 mm
- net D5: track 20.6 -> 0.00 mm
- net A5: track 19.9 -> 0.00 mm
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Other:
- board size 69.2 x 53.4 mm -> 68.6 x 53.3 mm
- board text removed: "0"
- board text removed: "1"
- board text removed: "10"
- board text removed: "11"
- board text removed: "12"
- board text removed: "13"
- board text removed: "2"
- board text removed: "3"
- board text removed: "3v"
- board text removed: "4"
- board text removed: "5"
- board text removed: "5v"
- board text removed: "6"
- board text removed: "7"
- board text removed: "8"
- board text removed: "9"
- board text removed: "ARef"
- board text removed: "Analog In"
- board text removed: "Digital I/O"
- board text removed: "Gnd"
- board text removed: "RST"
- board text removed: "Vin"
- board text removed: "gnd"

Commit message: ajout listes composants
Routing:
- net 12V: track 83.4 -> 84.0 mm
Other:
- board text added: "Batterie"
- board text added: "CAN"
Changed lines of the file:
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@@
 <board>
 <plain>
+<text x="1.905" y="32.7025" size="1.27" layer="25">Batterie</text>
+<text x="1.905" y="48.895" size="1.27" layer="25">CAN</text>
 </plain>
 <attributes>
@@
 <param name="srMinRoundness" value="0mil"/>
 <param name="srMaxRoundness" value="0mil"/>
-<param name="slThermalIsolate" value="10mil"/>
+<param name="slThermalIsolate" value="15mil"/>
 <param name="slThermalsForVias" value="0"/>
 <param name="dpMaxLengthDifference" value="10mm"/>
@@
 <contactref element="D1" pad="C"/>
 <contactref element="ALIM_ARDUINO" pad="2"/>
-<wire x1="10.795" y1="11.684" x2="17.145" y2="18.034" width="1.016" layer="1"/>
-<wire x1="17.145" y1="18.034" x2="21.59" y2="18.034" width="1.016" layer="1"/>
-<wire x1="16.256" y1="3.3655" x2="16.0655" y2="3.175" width="1.016" layer="1"/>
-<wire x1="16.0655" y1="3.175" x2="10.795" y2="3.175" width="1.016" layer="1"/>
-<wire x1="14.097" y1="25.8318" x2="21.59" y2="18.3388" width="1.016" layer="16"/>
+<wire x1="10.795" y1="11.684" x2="17.145" y2="18.034" width="1.27" layer="1"/>
+<wire x1="17.145" y1="18.034" x2="21.59" y2="18.034" width="1.27" layer="1"/>
+<wire x1="16.256" y1="3.3655" x2="16.0655" y2="3.175" width="1.27" layer="1"/>
+<wire x1="16.0655" y1="3.175" x2="10.795" y2="3.175" width="1.27" layer="1"/>
+<wire x1="14.097" y1="25.8318" x2="21.59" y2="18.3388" width="1.27" layer="16"/>
 <wire x1="21.59" y1="18.3388" x2="21.59" y2="18.034" width="1.016" layer="16"/>
 <contactref element="C4" pad="2"/>
@@
 <wire x1="21.59" y1="18.034" x2="21.86441875" y2="18.034" width="1.016" layer="16"/>
 <wire x1="21.86441875" y1="18.034" x2="21.95331875" y2="17.9451" width="1.016" layer="16"/>
-<wire x1="27.94" y1="24.13" x2="30.48" y2="21.59" width="1.016" layer="16"/>
-<wire x1="6.35" y1="3.175" x2="10.795" y2="3.175" width="1.016" layer="1"/>
-<wire x1="10.795" y1="11.684" x2="10.795" y2="3.175" width="1.016" layer="1"/>
+<wire x1="27.94" y1="24.13" x2="30.48" y2="21.59" width="1.27" layer="16"/>
+<wire x1="6.35" y1="3.175" x2="10.795" y2="3.175" width="1.27" layer="1"/>
+<wire x1="10.795" y1="11.684" x2="10.795" y2="3.175" width="1.27" layer="1"/>
 <contactref element="C3" pad="1"/>
 <contactref element="PS1" pad="1"/>
-<wire x1="30.48" y1="13.97" x2="41.91" y2="13.97" width="1.016" layer="1"/>
-<wire x1="41.91" y1="13.97" x2="48.22" y2="7.66" width="1.016" layer="1"/>
-<wire x1="30.48" y1="21.59" x2="30.48" y2="17.9451" width="1.016" layer="16"/>
-<wire x1="30.48" y1="17.78" x2="30.48" y2="13.97" width="1.016" layer="16"/>
-<wire x1="21.95331875" y1="17.9451" x2="30.48" y2="17.9451" width="1.016" layer="16"/>
-<wire x1="30.48" y1="17.9451" x2="30.48" y2="17.78" width="0" layer="19" extent="16-16"/>
+<wire x1="30.48" y1="13.97" x2="41.91" y2="13.97" width="1.27" layer="1"/>
+<wire x1="41.91" y1="13.97" x2="48.22" y2="7.66" width="1.27" layer="1"/>
+<wire x1="30.48" y1="21.59" x2="30.48" y2="17.9451" width="1.27" layer="16"/>
+<wire x1="30.48" y1="17.9451" x2="30.3911" y2="18.034" width="1.27" layer="16"/>
+<wire x1="30.3911" y1="18.034" x2="21.59" y2="18.034" width="1.27" layer="16"/>
+<wire x1="30.48" y1="17.9451" x2="30.48" y2="13.97" width="1.27" layer="16"/>
 </signal>
 <signal name="N$4">
 <contactref element="D1" pad="A"/>
 <contactref element="R20" pad="2"/>
-<wire x1="26.416" y1="3.3655" x2="29.21" y2="6.1595" width="1.016" layer="1"/>
-<wire x1="29.21" y1="6.1595" x2="29.21" y2="6.985" width="1.016" layer="1"/>
+<wire x1="26.416" y1="3.3655" x2="29.21" y2="6.1595" width="1.27" layer="1"/>
+<wire x1="29.21" y1="6.1595" x2="29.21" y2="6.985" width="1.27" layer="1"/>
 </signal>
 <signal name="N$1">
 <contactref element="J5" pad="1"/>
 <contactref element="F1" pad="1"/>
-<wire x1="6.223" y1="38.989" x2="14.097" y2="46.863" width="1.016" layer="1"/>
-<wire x1="14.097" y1="46.863" x2="14.097" y2="50.8762" width="1.016" layer="1"/>
+<wire x1="6.223" y1="38.989" x2="14.097" y2="46.863" width="1.27" layer="1"/>
+<wire x1="14.097" y1="46.863" x2="14.097" y2="50.8762" width="1.27" layer="1"/>
 </signal>
 <signal name="N$3">
 <contactref element="PS1" pad="5"/>
 <contactref element="C5" pad="1"/>
-<wire x1="35.52" y1="27.98" x2="34.29" y2="29.21" width="1.016" layer="1"/>
-<wire x1="34.29" y1="29.21" x2="30.48" y2="29.21" width="1.016" layer="1"/>
+<wire x1="35.52" y1="27.98" x2="34.29" y2="29.21" width="1.27" layer="1"/>
+<wire x1="34.29" y1="29.21" x2="30.48" y2="29.21" width="1.27" layer="1"/>
 </signal>
 <signal name="N$5">
@@
 <contactref element="QUARTZ_16_MHZ" pad="1"/>
 <contactref element="IC2" pad="8"/>
-<wire x1="55.4938" y1="32.2685375" x2="54.5314625" y2="31.3062" width="0.6096" layer="1"/>
-<wire x1="55.88" y1="33.425" x2="55.4938" y2="33.0388" width="0.6096" layer="1"/>
-<wire x1="55.4938" y1="33.0388" x2="55.4938" y2="32.2685375" width="0.6096" layer="1"/>
+<wire x1="55.8113" y1="32.5860375" x2="54.5314625" y2="31.3062" width="0.6096" layer="1"/>
+<wire x1="55.88" y1="33.425" x2="55.8113" y2="33.3563" width="0.6096" layer="1"/>
+<wire x1="55.8113" y1="33.3563" x2="55.8113" y2="32.5860375" width="0.6096" layer="1"/>
 <wire x1="54.5314625" y1="31.3062" x2="47.0685375" y2="31.3062" width="0.6096" layer="1"/>
 <wire x1="47.0685375" y1="31.3062" x2="43.18" y2="35.1947375" width="0.6096" layer="1"/>
@@
 <contactref element="C4" pad="1"/>
 <contactref element="PS1" pad="3"/>
-<wire x1="30.48" y1="24.13" x2="49.45" y2="24.13" width="0.6096" layer="1"/>
+<wire x1="30.48" y1="24.13" x2="49.45" y2="24.13" width="1.27" layer="1"/>
 <contactref element="J1" pad="5"/>
-<wire x1="55.88" y1="24.13" x2="55.84" y2="24.17" width="0.6096" layer="16"/>
-<wire x1="55.88" y1="18.415" x2="61.595" y2="12.7" width="2.54" layer="16"/>
-<wire x1="61.595" y1="12.7" x2="64.77" y2="12.7" width="2.54" layer="16"/>
-<wire x1="55.88" y1="24.13" x2="55.88" y2="18.415" width="2.54" layer="16"/>
-<wire x1="55.88" y1="24.13" x2="55.88" y2="27.94" width="2.54" layer="16"/>
-<wire x1="49.45" y1="24.13" x2="53.3" y2="27.98" width="0.6096" layer="1"/>
-<wire x1="53.3" y1="27.98" x2="55.84" y2="27.98" width="0.6096" layer="1"/>
+<wire x1="64.77" y1="12.7" x2="61.595" y2="12.7" width="2.54" layer="16"/>
+<wire x1="49.45" y1="24.13" x2="53.3" y2="27.98" width="1.27" layer="1"/>
+<wire x1="53.3" y1="27.98" x2="55.84" y2="27.98" width="1.27" layer="1"/>
 <wire x1="55.84" y1="27.98" x2="58.6688" y2="30.8088" width="0.6096" layer="1"/>
 <wire x1="58.6688" y1="30.8088" x2="58.6688" y2="35.2164625" width="0.6096" layer="1"/>
 <wire x1="37.625" y1="43.18" x2="46.585" y2="43.18" width="0.6096" layer="1"/>
 <wire x1="46.585" y1="43.18" x2="46.99" y2="42.775" width="0.6096" layer="1"/>
-<wire x1="55.84" y1="27.98" x2="55.88" y2="27.94" width="0" layer="19" extent="16-16"/>
+<wire x1="55.84" y1="18.455" x2="55.84" y2="27.98" width="2.54" layer="16"/>
+<wire x1="61.595" y1="12.7" x2="55.84" y2="18.455" width="2.54" layer="16"/>
 </signal>
 <signal name="N$7">
